File: PCB-IOBoard/AMP2-IO.brd (EAGLE design)
At the start: 100.4 x 80 mm, 37 parts, among them IC3 REG1117, IC4 REG1117

Commit message: Getting somewhere.
Parts:
- removed SV1: (no value), con-lsta:FE10-2
- removed SV2: (no value), con-lsta:FE08
- added C18, C19: 100u, rcl:153CLV-0807
- added C20: 100n, rcl:C0805K
- added C21, C22: 12p, rcl:C0805K
- added H1, H2, H3, H4: MOUNT-HOLE3.2, holes:3,2
- added Q2: 12.288, crystal:CTS406
- added R10, R11, R9: 47, rcl:R0805W
- added R6, R8: 4.02k, rcl:R0805W
- added R7: 1k, rcl:R0805W
- added SJ1: (no value), jumper:SJ
- added SV3: (no value), con-lsta:FE08
- added SV4: (no value), con-lsta:FE10-2
- C3, C4: device rcl:153CLV-1010 -> rcl:153CLV-0807
- C5: value (none) -> 100n
- L1: device rcl:L5650M -> rcl:L4532P
- L2: device rcl:L5650M -> rcl:L4532M
- moved C5 64.0 mm to (94.7, 32.0)
- moved IC3 43.4 mm to (53.6, 7.37), turned to 180 degrees
- moved C3 42.7 mm to (62.5, 7.37), turned to 90 degrees
- moved U$4 36.7 mm to (31.2, 30.0), turned to 0 degrees
- moved C4 32.0 mm to (45.0, 7.37), turned to 90 degrees
- moved C15 31.3 mm to (25.4, 49.5), turned to 0 degrees
- moved C14 30.9 mm to (25.4, 53.1), turned to 0 degrees
- moved IC4 24.2 mm to (25.9, 7.37), turned to 180 degrees
- moved L2 22.1 mm to (15.0, 17.8), turned to 90 degrees
- moved U$1 22.0 mm to (62.2, 33.5)
- moved R3 18.3 mm to (72.6, 44.2)
- moved U$2 14.2 mm to (31.8, 44.2)
- moved R1 14.0 mm to (96.8, 58.4), turned to 270 degrees
- moved U$6 13.1 mm to (45.7, 39.1), turned to 90 degrees
- moved R5 11.2 mm to (31.0, 51.3)
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Connections:
- new net +5V: C18.+, IC4.3, SV3.3, SV3.4
- new net ADR/FAULT: SV4.1
- new net GND1: SV3.7, SV3.8
- new net LRCLK: R9.1, SV4.13
- new net MCLK: U$1.10, U$3.15
- new net N$20: C21.2, Q2.1, U$1.2
- new net N$21: R6.1, U$1.15
- new net N$22: R7.1, U$1.19
- new net N$23: R8.1, U$1.18
- new net N$24: C22.2, Q2.3, U$1.1
- new net N$25: R11.2, U$1.12
- new net N$26: R10.2, U$1.13
- new net N$27: R9.2, U$1.14
- new net PDN: SV4.3
- new net SCL: SV4.17, U$4.3
- new net SCLK: R10.1, SV4.11
- new net SDA: SV4.15, U$4.4
- new net SDIN: R11.1, SV4.7
- new net SDOUT: SV4.9
- net +12V: now also SV3.1, SV3.2
- net +3V3: now also C19.+, C5.1, SV3.5, SV3.6, U$3.17, U$3.19, U$3.20, U$3.7
- net A5V: now also C20.1
- net AGND: now also C20.2, SJ1.1
- net GND: now also C18.-, C19.-, C21.1, C22.1, C5.2, R6.2, R7.2, R8.2, SJ1.2, SV4.10, SV4.12, SV4.14, SV4.16, SV4.18, SV4.20, SV4.6, SV4.8, U$3.16, U$3.18, U$3.8
- net SW_BCK: now also U$1.8
- net SW_SCLK: no longer U$1.8
Routing:
- net N$2: track 0.00 -> 24.4 mm
- net N$1: track 0.00 -> 16.7 mm
- net N$25: track 0.00 -> 12.8 mm
- net N$26: track 0.00 -> 11.0 mm
- net N$27: track 0.00 -> 10.2 mm
- net LRCLK: track 0.00 -> 6.75 mm
- net SDIN: track 0.00 -> 6.60 mm
- net SCLK: track 0.00 -> 6.60 mm
- net N$21: track 0.00 -> 2.52 mm
- net N$23: track 0.00 -> 2.48 mm
- net N$22: track 0.00 -> 2.34 mm
- net N$4: track 17.5 -> 18.3 mm
- added copper zone on layer 16, net AGND

Commit message: Added Ext Headers, TORX, ... not complete yet.
Parts:
- added C23: 10u, rcl:153CLV-0807
- added C24: 100n, rcl:C0805K
- added C25: 4.7n, rcl:C0805K
- added D1, D2: (no value), diode:SMB
- added EXT1, EXT2: (no value), con-lsta:FE08
- added IC1: 7404D, 74xx-eu:SO14
- added IC2: R-78E-0.5, linear:TO220V
- added L3: (no value), rcl:L4532P
- added L5: 10uH, inductors:DR125
- added SJ2: (no value), jumper:SJ
- added SV1: (no value), con-lsta:FE05-1
- added U$7: TORX135X, AMP2-ICs:TORX135X
- added X3: MKDSN1,5/2-5,08, con-phoenix-508:MKDSN1,5/2-5,08
- C18: value 100u -> 10u
- C4: value (none) -> 10u
- R3: value 0 -> 680; device rcl:R1206W -> rcl:R0805W
- moved R3 57.6 mm to (19.1, 65.3), turned to 0 degrees
- moved C4 50.0 mm to (93.5, 19.6), turned to 180 degrees
- moved L1 45.2 mm to (85.1, 17.3), turned to 90 degrees
- moved C3 38.4 mm to (93.5, 30.0), turned to 180 degrees
- moved IC3 34.7 mm to (80.5, 29.2), turned to 90 degrees
- moved L2 34.0 mm to (31.5, 47.5), turned to 180 degrees
- moved R2 30.8 mm to (55.9, 60.7)
- moved C5 25.9 mm to (69.6, 38.1), turned to 180 degrees
- moved C2 20.6 mm to (61.2, 59.4)
- moved C19 18.4 mm to (15.0, 25.4), turned to 0 degrees
- moved IC4 18.0 mm to (26.4, 25.4), turned to 270 degrees
- moved C18 17.8 mm to (17.0, 8.13)
- moved U$3 17.8 mm to (70.9, 43.9)
- moved C16 13.5 mm to (44.5, 58.9)
- moved R5 13.3 mm to (41.1, 59.9)
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Connections:
- removed net +5V: C18.+, IC4.3, SV3.3, SV3.4
- new net +7V: C18.+, IC2.3, IC4.3, L1.1
- new net BCLK_EX1: EXT1.6, U$5.2
- new net BCLK_EX2: EXT2.6, U$5.4
- new net DOUT_EX1: EXT1.4, U$6.2
- new net DOUT_EX2: EXT2.4, U$6.4
- new net ERNIE: D1.A, L5.2
- new net GP6: EXT1.2, U$4.16
- new net GP7: EXT2.2, U$4.17
- new net HORST: L5.1, X3.2
- new net LRCK_EX1: EXT1.5, U$6.15
- new net LRCK_EX2: EXT2.5, U$6.11
- new net N$28: C24.1, L3.2, U$7.3
- new net N$29: IC1.1, IC1.4
- new net N$30: C23.+, D1.C, D2.C, IC2.1
- new net N$31: C25.1, R3.1, SPDIF.2
- new net N$32: C25.2, IC1.3
- new net SCLK_EX1: EXT1.7, U$5.15
- new net SCLK_EX2: EXT2.7, U$5.11
- net +12V: now also D2.A; no longer L1.1
- net +3V3: now also EXT1.8, EXT2.8, IC1.14, U$4.1; no longer SV3.5, SV3.6
- net AGND: now also C24.2, IC1.11, IC1.13, IC1.5, IC1.7, IC1.9, L3.1, SJ2.1, U$7.2
- net GND: now also C23.-, EXT1.1, EXT1.3, EXT2.1, EXT2.3, IC2.2, SJ2.2, SV1.1, U$4.20, U$7.5, U$7.6, X3.1; no longer R3.1
- net N$19: now also U$7.1
- net SCL: now also SV1.2
- net SDA: now also SV1.3
Routing:
- net N$2: track 24.4 -> 0.00 mm
- net N$4: track 18.3 -> 0.00 mm
- net N$1: track 16.7 -> 0.00 mm
- net N$3: track 15.9 -> 0.00 mm
- net N$25: track 12.8 -> 0.00 mm
- net N$26: track 11.0 -> 0.00 mm
- net N$27: track 10.2 -> 0.00 mm
- net LRCLK: track 6.75 -> 0.00 mm
- net SDIN: track 6.60 -> 0.00 mm
- net SCLK: track 6.60 -> 0.00 mm
- net N$21: track 2.52 -> 0.00 mm
- net N$23: track 2.48 -> 0.00 mm
- net N$22: track 2.34 -> 0.00 mm
Other:
- board text added: "1"
- board text added: "3.3V"
- board text added: "9-24V"
- board text added: "BCLK"
- board text added: "DOUT"
- board text added: "GND"
- board text added: "GP6"
- board text added: "GP7"
- board text added: "LRCK"
- board text added: "SCL"
- board text added: "SCLK"
- board text added: "SDA"

Commit message: Autorouted and Manual Layout
Parts:
- added C26, C27: 100n, rcl:C0805K
- added D3: MBR0520LT, diode:SOD123
- added K2: GN210S03, relay:GN-S
- moved C7 20.8 mm to (68.6, 42.2), turned to 180 degrees
- moved C9 15.5 mm to (68.8, 39.1), turned to 180 degrees
- moved C3 15.3 mm to (92.2, 45.2)
- moved C14 14.1 mm to (42.2, 60.7), turned to 0 degrees
- moved C15 9.67 mm to (41.9, 57.4), turned to 0 degrees
- moved C4 9.27 mm to (91.9, 28.7)
- moved IC3 7.98 mm to (81.8, 37.1), turned to 180 degrees
- moved IC4 7.89 mm to (18.8, 27.4)
- moved L2 7.54 mm to (37.8, 51.6), turned to 90 degrees
- moved C19 7.23 mm to (12.7, 18.5), turned to 90 degrees
- moved U$2 5.79 mm to (45.7, 51.6)
- moved C17 5.73 mm to (50.0, 59.7)
- moved R5 5.73 mm to (46.7, 58.7)
- moved C16 5.73 mm to (50.0, 57.7)
- moved U$3 5.09 mm to (70.6, 49.0)
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Connections:
- new net N$33: K2.5, U$7.1
- new net N$34: IC1.2, K2.7
- new net N$35: D3.C, IC1.10, IC1.12, IC1.6, IC1.8, K2.8
- new net RELAIS: IC1.11, IC1.13, IC1.5, IC1.9, U$4.12
- net +3V3: now also C26.1, C27.1, U$1.17, U$1.3
- net AGND: no longer IC1.11, IC1.13, IC1.5, IC1.7, IC1.9
- net GND: now also C26.2, C27.2, D3.A, IC1.7, K2.1, U$1.16, U$1.4
- net N$19: now also K2.6; no longer U$7.1
Routing:
- net +3V3: track 0.00 -> 151.7 mm, vias 0 -> 15
- net GND: track 0.00 -> 117.8 mm, vias 0 -> 26
- net +7V: track 0.00 -> 99.4 mm
- net SCL: track 0.00 -> 88.7 mm, vias 0 -> 3
- net SDA: track 0.00 -> 87.3 mm, vias 0 -> 3
- net DOUT_EX1: track 0.00 -> 56.0 mm, vias 0 -> 2
- net BCLK_EX1: track 0.00 -> 51.7 mm, vias 0 -> 1
- net DOUT_EX2: track 0.00 -> 51.7 mm, vias 0 -> 2
- net BCLK_EX2: track 0.00 -> 49.2 mm, vias 0 -> 2
- net LRCK_EX1: track 0.00 -> 48.9 mm, vias 0 -> 1
- net +12V: track 0.00 -> 45.6 mm
- net N$35: track 0.00 -> 43.6 mm
- net SCLK_EX1: track 0.00 -> 42.4 mm, vias 0 -> 1
- net LRCK_EX2: track 0.00 -> 40.1 mm, vias 0 -> 2
- net SCLK_EX2: track 0.00 -> 39.8 mm, vias 0 -> 2
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- added copper zone on layer 1, net +3V3
- added copper zone on layer 16, net +3V3
- added copper zone on layer 1, net A5V

Commit message: Routed.
Parts:
- added FS1, FS2, POWER, RX_ERROR, SRCUNLOCK: (no value), led:CHIPLED_0805
- added R12, R13, R14, R15, R16, R20: 1k, rcl:R0805W
- added R17: 47k, rcl:R0805W
- added R18: 2.2k, rcl:R0805W
- added R19: 4.02k, rcl:R0805W
- added R21: open, rcl:R0805W
- added SRC_BYPASS: (no value), jumper:JP1
- C25: value 4.7n -> 10n
- IC2: value R-78E-0.5 -> R-78E9.0-0.5
- R3: value 680 -> 75
- R8: value 4.02k -> 8.04k
- moved C26 12.5 mm to (11.2, 57.7)
- moved D3 4.34 mm to (23.9, 57.4), turned to 270 degrees
- moved IC1 1.78 mm to (17.5, 56.6)
- moved L3 0.25 mm to (50.8, 71.4), turned to 270 degrees
- moved C24 0.25 mm to (46.2, 71.1), turned to 90 degrees
Connections:
- removed net PDN: SV4.3
- new net ERROR: R15.2, U$2.27, U$4.15
- new net FSOUT0: R14.2, U$2.2, U$4.14
- new net FSOUT1: R13.2, U$2.3, U$4.13
- new net N$36: POWER.A, R12.1
- new net N$37: FS1.A, R13.1
- new net N$38: FS2.A, R14.1
- new net N$39: R15.1, RX_ERROR.A
- new net N$40: R16.1, SRCUNLOCK.A
- new net N$41: R19.2, SRC_BYPASS.1, U$1.6
- new net N$42: R20.1, R21.2, U$4.5
- new net SRC_UNLOCK: R16.2, U$1.20, U$4.16
- net +3V3: now also R12.2, R21.1, SRC_BYPASS.2
- net AGND: no longer C24.2, L3.1, R3.2, SPDIF.1, SPDIF.1@1, SPDIF.1@2, U$7.2
- net GND: now also C24.2, FS1.C, FS2.C, IC1.5, L3.1, POWER.C, R18.1, R19.1, R20.2, R3.2, RX_ERROR.C, SPDIF.1, SPDIF.1@1, SPDIF.1@2, SRCUNLOCK.C, U$1.11, U$7.2
- net GP6: no longer U$4.16
- net GP7: now also U$4.12; no longer U$4.17
- net N$29: now also R17.2, R18.2
- net N$32: now also R17.1
- net N$35: no longer IC1.6
- net RELAIS: now also U$4.17; no longer IC1.5, U$4.12
- net RESET: now also SV4.3, U$1.5
Routing:
- net SRC_UNLOCK: track 0.00 -> 95.7 mm, vias 0 -> 4
- net RESET: track 0.00 -> 60.6 mm, vias 0 -> 5
- net GND: track 117.8 -> 66.6 mm, vias 26 -> 52
- net GP6: track 36.2 -> 0.00 mm
- net N$41: track 0.00 -> 33.0 mm, vias 0 -> 2
- net ERROR: track 0.00 -> 32.0 mm, vias 0 -> 2
- net FSOUT0: track 0.00 -> 22.3 mm
- net FSOUT1: track 0.00 -> 18.5 mm
- net N$35: track 43.6 -> 28.1 mm
- net N$42: track 0.00 -> 12.6 mm, vias 0 -> 2
- net RELAIS: track 33.3 -> 40.9 mm
- net N$29: track 7.63 -> 12.5 mm
- net GP7: track 22.3 -> 26.9 mm
- net N$32: track 9.16 -> 6.14 mm, vias 2 -> 0
- net N$40: track 0.00 -> 2.22 mm
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- added copper zone on layer 16, net A5V
Other:
- board text added: "5x"

Commit message: Switched to SRC4192
Parts:
- removed C22: 12p, rcl:C0805K
- removed Q2: 12.288, crystal:CTS406
- removed R7: 1k, rcl:R0805W
- removed R8: 8.04k, rcl:R0805W
- added Q4: 12.288, crystal-geyer_V1_0:7.0X5.0_KXO-82-TCXO
- C18, C19, C23, C3, C4: device rcl:153CLV-0807 -> rcl:CT6032
- C21: value 12p -> 100n
- C25: value 10n -> 100n
- R6: value 4.02k -> 1k
- U$1: value CS8421 -> SRC4192; device AMP2-ICs:TSSOP20 -> AMP2-ICs:SSOP28BU
- moved R6 54.8 mm to (11.2, 55.9)
- moved C21 17.4 mm to (65.5, 40.4)
- moved C26 13.3 mm to (23.9, 53.6), turned to 0 degrees
- moved C18 3.14 mm to (14.0, 8.89), turned to 270 degrees
- moved C7 3.05 mm to (71.6, 42.2)
- moved C9 3.05 mm to (71.9, 39.1)
- moved C5 2.75 mm to (67.3, 36.8), turned to 90 degrees
- moved C23 2.59 mm to (67.8, 10.7)
- moved C4 2.55 mm to (92.2, 31.2), turned to 90 degrees
- moved C3 2.54 mm to (92.2, 42.7), turned to 270 degrees
- moved U$1 2.29 mm to (59.9, 33.5), turned to 270 degrees
- moved R4 2.17 mm to (71.4, 55.1)
- moved D2 2.05 mm to (58.2, 12.7), turned to 180 degrees
- moved C6 1.83 mm to (67.1, 57.7)
- moved C12 1.63 mm to (72.9, 60.5), turned to 0 degrees
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- renumbered SRCUNLOCK to SRCLOCK
Connections:
- net HORST renamed VIN
- net N$30 renamed VIN2
- removed net N$20: C21.2, Q2.1, U$1.2
- removed net N$21: R6.1, U$1.15
- removed net N$22: R7.1, U$1.19
- removed net N$23: R8.1, U$1.18
- removed net N$24: C22.2, Q2.3, U$1.1
- removed net SRC_UNLOCK: R16.2, U$1.20, U$4.16
- new net GND/NC: Q4.1
- new net SRC_LOCK: R16.2, U$1.14, U$1.15, U$4.16
- net +3V3: now also C21.1, Q4.4, U$1.10, U$1.19, U$1.22, U$1.26, U$1.7; no longer U$1.17, U$1.3
- net AGND: no longer C14.2, C15.2, C16.1, C17.1, U$2.23
- net GND: now also C14.2, C15.2, C16.1, C17.1, C21.2, Q4.2, U$1.1, U$1.12, U$1.17, U$1.18, U$1.20, U$1.21, U$1.27, U$1.28, U$1.8, U$2.23; no longer C21.1, C22.1, R7.2, R8.2, U$1.4
- net MCLK: now also Q4.3, U$1.2; no longer U$1.10
- net N$25: now also U$1.23; no longer U$1.12
- net N$26: now also U$1.25; no longer U$1.13
- net N$27: now also U$1.24; no longer U$1.14
- net N$41: now also U$1.9; no longer U$1.6
- net RELAIS: now also R6.1
- net RESET: now also U$1.13; no longer U$1.5
- net SW_BCK: now also U$1.5; no longer U$1.8
- net SW_DOUT: now also U$1.4; no longer U$1.9
- net SW_LRCK: now also U$1.6; no longer U$1.7
Routing:
- net SRC_UNLOCK: track 95.7 -> 0.00 mm, vias 4 -> 0
- net SRC_LOCK: track 0.00 -> 79.3 mm, vias 0 -> 6
- net SW_DOUT: track 39.2 -> 6.79 mm, vias 2 -> 0
- net +3V3: track 151.2 -> 175.6 mm, vias 28 -> 32
- net SW_LRCK: track 32.8 -> 14.0 mm, vias 2 -> 1
- net N$9: track 30.3 -> 41.8 mm, vias 2 -> 4
- net N$20: track 9.38 -> 0.00 mm
- net N$41: track 33.0 -> 24.0 mm
- net N$24: track 7.67 -> 0.00 mm
- net +7V: track 99.3 -> 105.0 mm
- net MCLK: track 26.4 -> 20.8 mm, vias 2 -> 0
- net RELAIS: track 40.9 -> 45.7 mm
- net N$5: track 37.9 -> 41.2 mm
- net A5V: track 34.8 -> 37.7 mm
- net N$7: track 32.1 -> 29.4 mm, vias 4 -> 2
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Other:
- board text added: "+"
- board text added: "-"

Commit message: Tuning..
Routing:
- net AGND: track 12.3 -> 7.43 mm, vias 27 -> 35
- net GND: vias 182 -> 193
Changed lines of the file:
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@@
 <?xml version="1.0" encoding="utf-8"?>
 <!DOCTYPE eagle SYSTEM "eagle.dtd">
-<eagle version="9.5.2">
+<eagle version="9.6.2">
 <drawing>
 <settings>
@@
 <via x="35.56" y="66.802" extent="1-16" drill="0.35"/>
 <via x="35.56" y="68.326" extent="1-16" drill="0.35"/>
+<via x="49.276" y="52.578" extent="1-16" drill="0.35"/>
+<via x="40.132" y="54.102" extent="1-16" drill="0.35"/>
+<via x="52.324" y="55.626" extent="1-16" drill="0.35"/>
+<via x="38.1" y="39.624" extent="1-16" drill="0.35"/>
+<via x="40.132" y="41.402" extent="1-16" drill="0.35"/>
+<via x="47.752" y="35.56" extent="1-16" drill="0.35"/>
+<via x="46.482" y="35.306" extent="1-16" drill="0.35"/>
+<via x="46.482" y="33.274" extent="1-16" drill="0.35"/>
+<via x="46.482" y="32.004" extent="1-16" drill="0.35"/>
+<via x="47.752" y="30.48" extent="1-16" drill="0.35"/>
+<via x="49.53" y="31.242" extent="1-16" drill="0.35"/>
 </signal>
 <signal name="N$1">
@@
 <wire x1="84.0486" y1="40.2336" x2="91.3384" y2="40.2336" width="1.016" layer="1"/>
 <wire x1="91.3384" y1="40.2336" x2="91.44" y2="40.132" width="0.3048" layer="1"/>
-<wire x1="95.252" y1="43.944" x2="92.202" y2="40.172" width="1.016" layer="1"/>
 <via x="54.61" y="56.896" extent="1-16" drill="0.35"/>
 <via x="54.61" y="63.246" extent="1-16" drill="0.35"/>
@@
 <via x="64.516" y="60.452" extent="1-16" drill="0.35"/>
 <via x="63.5" y="58.674" extent="1-16" drill="0.35"/>
+<via x="53.848" y="55.626" extent="1-16" drill="0.35"/>
+<via x="54.61" y="54.61" extent="1-16" drill="0.35"/>
+<via x="53.848" y="53.34" extent="1-16" drill="0.35"/>
+<via x="54.61" y="52.578" extent="1-16" drill="0.35"/>
+<via x="55.88" y="51.816" extent="1-16" drill="0.35"/>
+<via x="56.642" y="51.054" extent="1-16" drill="0.35"/>
+<via x="57.658" y="52.07" extent="1-16" drill="0.35"/>
+<via x="58.674" y="53.086" extent="1-16" drill="0.35"/>
 </signal>
 <signal name="A5V">
@@
 <wire x1="70.96125" y1="52.22875" x2="70.96125" y2="51.1175" width="0.254" layer="1"/>
 <wire x1="70.96125" y1="52.22875" x2="70.929" y2="52.324" width="0.254" layer="1"/>
-<wire x1="82.07375" y1="44.67225" x2="87.59825" y2="44.67225" width="0.3048" layer="1"/>
-<wire x1="87.59825" y1="44.67225" x2="88.138" y2="45.212" width="0.3048" layer="1"/>
-<wire x1="88.138" y1="45.212" x2="92.202" y2="45.172" width="0.3048" layer="1"/>
+<wire x1="82.07375" y1="44.67225" x2="87.59825" y2="44.67225" width="1.016" layer="1"/>
+<wire x1="87.59825" y1="44.67225" x2="88.138" y2="45.212" width="1.016" layer="1"/>
+<wire x1="88.138" y1="45.212" x2="92.202" y2="45.172" width="1.016" layer="1"/>
 <polygon width="0.3048" layer="1" rank="5">
 <vertex x="75.692" y="46.228"/>
@@
 <wire x1="43.97375" y1="42.70375" x2="43.97375" y2="40.3225" width="0.254" layer="16"/>
 <wire x1="43.02125" y1="43.65625" x2="43.97375" y2="42.70375" width="0.254" layer="16"/>
-<wire x1="20.32" y1="43.65625" x2="43.02125" y2="43.65625" width="0.254" layer="16"/>
-<wire x1="7.62" y1="56.35625" x2="20.32" y2="43.65625" width="0.254" layer="16"/>
-<wire x1="6.6675" y1="56.35625" x2="7.62" y2="56.35625" width="0.254" layer="16"/>
+<wire x1="20.574" y1="43.65625" x2="43.02125" y2="43.65625" width="0.254" layer="16"/>
+<wire x1="7.874" y1="56.35625" x2="20.574" y2="43.65625" width="0.254" layer="16"/>
+<wire x1="6.6675" y1="56.35625" x2="7.874" y2="56.35625" width="0.254" layer="16"/>
 <wire x1="44.60875" y1="38.25875" x2="44.727" y2="38.253" width="0.254" layer="1"/>
 <wire x1="6.6675" y1="56.35625" x2="6.604" y2="56.388" width="0.254" layer="16"/>
@@
 <wire x1="48.41875" y1="43.4975" x2="48.41875" y2="40.48125" width="0.254" layer="1"/>
 <wire x1="48.5775" y1="43.65625" x2="48.41875" y2="43.4975" width="0.254" layer="1"/>
-<wire x1="46.736" y1="45.49775" x2="48.5775" y2="43.65625" width="0.254" layer="16"/>
-<wire x1="39.90975" y1="45.49775" x2="46.736" y2="45.49775" width="0.254" layer="16"/>
+<wire x1="48.3235" y1="43.65625" x2="46.99" y2="44.98975" width="0.254" layer="16"/>
+<wire x1="48.3235" y1="43.65625" x2="48.5775" y2="43.65625" width="0.254" layer="16"/>
+<wire x1="39.90975" y1="45.49775" x2="40.41775" y2="44.98975" width="0.254" layer="16"/>
+<wire x1="46.99" y1="44.98975" x2="40.41775" y2="44.98975" width="0.254" layer="16"/>
 <wire x1="39.90975" y1="45.49775" x2="39.90975" y2="42.672" width="0.254" layer="1"/>
 <wire x1="39.90975" y1="42.672" x2="35.78225" y2="38.5445" width="0.254" layer="1"/>

Commit message: 603 packs and some other stuff. Changed MCLK to 24.576 needed by DIR9001 for FS detection.
Parts:
- added OX1: TORX173, toshiba:TORX173
- C11, C13, C15, C16, C17, C20, C21, C24, C25, C26, C27, C5, C6, C7: device rcl:C0805K -> rcl:C0603
- C19: value 100u -> 10u
- C3: value (none) -> 10u
- L1, L3: value (none) -> 220uH; device rcl:L4532P -> rcl:L4532M
- L2: value (none) -> 220uH
- Q4: value 12.288 -> 24.576
- R1, R10, R11, R17, R18, R2, R21, R3, R5, R9: device rcl:R0805W -> rcl:R0603
- R12, R13, R14, R15, R16, R20, R4, R6: value 1k -> 2.2k; device rcl:R0805W -> rcl:R0603
- R19: value 4.02k -> 2.2k; device rcl:R0805W -> rcl:R0603
Connections:
- net +3V3: now also U$1.27, U$2.28
- net GND: now also OX1.2, OX1.4, OX1.5, OX1.6; no longer U$1.27, U$2.28
- net MCLK: now also U$2.8
- net N$28: now also OX1.3
- net N$33: now also OX1.1
Routing:
- net MCLK: track 20.8 -> 42.4 mm, vias 0 -> 2
- net +3V3: track 175.6 -> 182.5 mm
- net GND: track 64.7 -> 58.2 mm
- net N$28: track 12.1 -> 15.3 mm
- net N$11: track 20.5 -> 23.2 mm
- net N$33: track 9.55 -> 11.2 mm
- net RESET: track 61.7 -> 62.3 mm

Commit message: Changed switching chipies to SN74CBT3253.
Parts:
- removed L5: 10uH, inductors:DR125
- U$5, U$6: value CD4052B -> SN74CBT3253
- moved U$5 13.6 mm to (45.0, 41.7), turned to 270 degrees
- moved U$6 7.41 mm to (45.0, 33.0), turned to 270 degrees
Connections:
- removed net VIN: L5.1, X3.2
- net BCLK_EX1: now also U$5.12; no longer U$5.2
- net BCLK_EX2: now also U$5.13; no longer U$5.4
- net DOUT_EX1: now also U$6.12; no longer U$6.2
- net DOUT_EX2: now also U$6.13; no longer U$6.4
- net ERNIE: now also X3.2; no longer L5.2
- net GND: now also U$5.1, U$5.15, U$6.1, U$6.15; no longer U$5.6, U$5.7, U$6.6, U$6.7
- net LRCK_EX1: now also U$6.4; no longer U$6.15
- net LRCK_EX2: now also U$6.3; no longer U$6.11
- net N$10: now also U$6.5; no longer U$6.14
- net N$11: now also U$6.11; no longer U$6.5
- net N$12: now also U$6.10; no longer U$6.1
- net N$6: now also U$5.6; no longer U$5.12
- net N$7: now also U$5.10; no longer U$5.1
- net N$8: now also U$6.6; no longer U$6.12
- net N$9: now also U$5.11; no longer U$5.5
- net SCLK_EX1: now also U$5.4; no longer U$5.15
- net SCLK_EX2: now also U$5.3; no longer U$5.11
- net SEL_A: now also U$5.14, U$6.14; no longer U$5.10, U$6.10
- net SEL_B: now also U$5.2, U$6.2; no longer U$5.9, U$6.9
- net SW_BCK: now also U$5.9; no longer U$5.3
- net SW_DOUT: now also U$6.9; no longer U$6.3
- net SW_LRCK: now also U$6.7; no longer U$6.13
- net SW_SCLK: now also U$5.7; no longer U$5.13
Routing:
- net BCLK_EX2: track 49.2 -> 88.8 mm, vias 2 -> 3
- net RESET: track 62.3 -> 90.5 mm, vias 2 -> 1
- net N$10: track 29.9 -> 52.4 mm
- net N$9: track 42.3 -> 22.9 mm, vias 4 -> 0
- net N$7: track 29.4 -> 10.8 mm
- net SCLK_EX1: track 42.7 -> 60.3 mm, vias 1 -> 3
- net BCLK_EX1: track 51.7 -> 65.5 mm, vias 1 -> 2
- net SEL_A: track 30.7 -> 43.8 mm
- net GND: track 58.2 -> 70.9 mm, vias 193 -> 192
- net SW_BCK: track 21.8 -> 10.1 mm, vias 2 -> 0
- net N$12: track 13.9 -> 25.0 mm, vias 0 -> 2
- net N$8: track 10.5 -> 21.0 mm, vias 0 -> 2
- net SRC_LOCK: track 79.5 -> 69.7 mm, vias 6 -> 5
- net DOUT_EX1: track 56.3 -> 64.6 mm
- net VIN: track 7.78 -> 0.00 mm
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Other:
- board text added: "@mb'2021"
- board text removed: "@mb'2020"
