File: PCB-IOBoard/AMP2-IO.brd (EAGLE design)
At the start: 100.4 x 80 mm, 89 parts, among them IC1 7404TS, IC2 R-78E6.5-0.5, IC3 REG1117, IC4 REG1117, K2 GN210S03, Q4 24.576, X3 MKDSN1,5/2-5,08

Commit message: Minor fixes.
Parts:
- OX1: device toshiba:TORX173 -> AMP2-ICs:TORX173
- moved U$7 0.51 mm to (36.6, 73.2)
Routing:
- net GND: track 72.8 -> 52.2 mm
Other:
- board text added: "Version: 0.1"
Changed lines of the file:
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@@
 <layer number="20" name="Dimension" color="24" fill="1" visible="yes" active="yes"/>
 <layer number="21" name="tPlace" color="7" fill="1" visible="yes" active="yes"/>
-<layer number="22" name="bPlace" color="7" fill="1" visible="no" active="yes"/>
+<layer number="22" name="bPlace" color="7" fill="1" visible="yes" active="yes"/>
 <layer number="23" name="tOrigins" color="15" fill="1" visible="yes" active="yes"/>
-<layer number="24" name="bOrigins" color="15" fill="1" visible="no" active="yes"/>
+<layer number="24" name="bOrigins" color="15" fill="1" visible="yes" active="yes"/>
 <layer number="25" name="tNames" color="7" fill="1" visible="yes" active="yes"/>
-<layer number="26" name="bNames" color="7" fill="1" visible="no" active="yes"/>
+<layer number="26" name="bNames" color="7" fill="1" visible="yes" active="yes"/>
 <layer number="27" name="tValues" color="7" fill="1" visible="yes" active="yes"/>
-<layer number="28" name="bValues" color="7" fill="1" visible="no" active="yes"/>
+<layer number="28" name="bValues" color="7" fill="1" visible="yes" active="yes"/>
 <layer number="29" name="tStop" color="7" fill="3" visible="no" active="yes"/>
 <layer number="30" name="bStop" color="7" fill="6" visible="no" active="yes"/>
@@
 <layer number="46" name="Milling" color="3" fill="1" visible="no" active="yes"/>
 <layer number="47" name="Measures" color="7" fill="1" visible="no" active="yes"/>
-<layer number="48" name="Document" color="7" fill="1" visible="yes" active="yes"/>
+<layer number="48" name="Document" color="7" fill="1" visible="no" active="yes"/>
 <layer number="49" name="Reference" color="7" fill="1" visible="no" active="yes"/>
 <layer number="50" name="dxf" color="7" fill="1" visible="no" active="yes"/>
@@
 <wire x1="0" y1="5.08" x2="5.08" y2="0" width="0" layer="20" curve="100"/>
 <text x="81.661" y="53.086" size="12.7" layer="26" font="vector" rot="MR0">mb'AMP2</text>
-<text x="37.338" y="47.625" size="1.6764" layer="26" rot="MR0">maker4makers.de</text>
-<text x="31.369" y="50.419" size="1.6764" layer="26" rot="MR0">@mb'2021</text>
+<text x="98.552" y="48.387" size="1.6764" layer="26" rot="MR0">maker4makers.de</text>
+<text x="98.425" y="51.943" size="1.6764" layer="26" rot="MR0">@mb'2021</text>
 <wire x1="-4.064" y1="51.054" x2="-4.064" y2="48.514" width="0.1524" layer="48"/>
 <wire x1="-4.064" y1="48.514" x2="-4.064" y2="46.736" width="0.1524" layer="48"/>
@@
 <wire x1="55.118" y1="24.13" x2="55.118" y2="14.732" width="0.4064" layer="25"/>
 <text x="54.61" y="14.986" size="1.778" layer="25" rot="R90">red</text>
+<text x="98.552" y="55.372" size="1.778" layer="26" rot="MR0">Version: 0.1</text>
 </plain>
 <attributes>
@@
 <attribute name="VALUE" x="60.198" y="48.6219" size="0.02" layer="28" rot="MR270"/>
 </element>
-<element name="U$7" library="AMP2-ICs" package="TORX135X" value="TORX135X" x="36.576" y="73.66" smashed="yes">
-<attribute name="MOUSER" value="757-TORX1355VF" x="36.576" y="73.66" size="1.778" layer="27" display="off"/>
-<attribute name="VALUE" x="41.402" y="73.279" size="1.27" layer="25" rot="R180"/>
+<element name="U$7" library="AMP2-ICs" package="TORX135X" value="TORX135X" x="36.576" y="73.152" smashed="yes">
+<attribute name="MOUSER" value="757-TORX1355VF" x="36.576" y="73.152" size="1.778" layer="27" display="off"/>
+<attribute name="VALUE" x="41.402" y="72.771" size="1.27" layer="25" rot="R180"/>
 </element>
 <element name="L3" library="rcl" library_urn="urn:adsk.eagle:library:334" package="L4532M" package3d_urn="urn:adsk.eagle:package:23483/2" value="220uH" x="50.8" y="71.374" smashed="yes" rot="R270">
@@
 <attribute name="SPICEPREFIX" value="R" x="13.716" y="54.864" size="1.778" layer="27" rot="R90" display="off"/>
 </element>
-<element name="OX1" library="toshiba" library_urn="urn:adsk.eagle:library:388" package="TORX173" package3d_urn="urn:adsk.eagle:package:28021/1" value="TORX173" x="36.576" y="70.866" smashed="yes">
+<element name="OX1" library="AMP2-ICs" package="TORX173" package3d_urn="urn:adsk.eagle:package:28021/1" value="TORX173" x="36.576" y="70.866" smashed="yes">
 <attribute name="MF" value="" x="36.576" y="70.866" size="1.778" layer="27" display="off"/>
 <attribute name="MPN" value="" x="36.576" y="70.866" size="1.778" layer="27" display="off"/>
@@
 <wire x1="8.1915" y1="60.67425" x2="6.604" y2="61.468" width="0.254" layer="1"/>
 <wire x1="6.604" y1="66.548" x2="6.604" y2="65.81775" width="0.254" layer="1"/>
-<wire x1="41.75125" y1="74.295" x2="31.4325" y2="74.295" width="0.254" layer="1"/>
-<wire x1="31.4325" y1="74.295" x2="31.376" y2="74.35" width="0.254" layer="1"/>
-<wire x1="41.75125" y1="74.295" x2="41.776" y2="74.35" width="0.254" layer="1"/>
+<wire x1="41.90890625" y1="74.13734375" x2="41.776" y2="73.842" width="0.254" layer="1"/>
 <wire x1="30.95625" y1="73.9775" x2="15.24" y2="73.9775" width="0.254" layer="1"/>
-<wire x1="31.27375" y1="74.295" x2="30.95625" y2="73.9775" width="0.254" layer="1"/>
-<wire x1="31.27375" y1="74.295" x2="31.376" y2="74.35" width="0.254" layer="1"/>
+<wire x1="31.376" y1="73.842" x2="31.029134375" y2="73.842" width="0.254" layer="1"/>
+<wire x1="31.029134375" y1="73.842" x2="30.95625" y2="73.9775" width="0.254" layer="1"/>
 <via x="33.274" y="33.274" extent="1-16" drill="0.35"/>
 <via x="19.304" y="34.036" extent="1-16" drill="0.35"/>
@@
 <wire x1="29.806" y1="23.876" x2="30.2625" y2="24.13" width="0.254" layer="1"/>
 <wire x1="30.2625" y1="24.13" x2="34.036" y2="24.13" width="0.254" layer="1"/>
-<wire x1="46.228" y1="71.97" x2="47.482" y2="73.374" width="0.3048" layer="1"/>
-<wire x1="47.482" y1="73.374" x2="50.8" y2="73.274" width="0.3048" layer="1"/>
-<wire x1="46.228" y1="71.97" x2="43.92625" y2="72.12" width="0.3048" layer="1"/>
-<wire x1="43.92625" y1="72.12" x2="41.75125" y2="74.295" width="0.3048" layer="1"/>
+<wire x1="41.90890625" y1="74.13734375" x2="41.75125" y2="74.295" width="0.3048" layer="1"/>
 <contactref element="Q4" pad="2"/>
 <contactref element="U$1" pad="21"/>
@@
 <via x="49.022" y="76.454" extent="1-16" drill="0.35"/>
 <via x="50.8" y="76.454" extent="1-16" drill="0.35"/>
-<via x="33.782" y="68.326" extent="1-16" drill="0.35"/>
+<via x="33.02" y="68.326" extent="1-16" drill="0.35"/>
 <via x="33.782" y="67.056" extent="1-16" drill="0.35"/>
 <via x="33.782" y="65.532" extent="1-16" drill="0.35"/>
@@
 <via x="40.132" y="54.102" extent="1-16" drill="0.35"/>
 <via x="52.324" y="55.626" extent="1-16" drill="0.35"/>
-<contactref element="OX1" pad="6"/>
-<contactref element="OX1" pad="5"/>
-<contactref element="OX1" pad="2"/>
-<contactref element="OX1" pad="4"/>
 <contactref element="U$5" pad="8"/>
 <contactref element="U$6" pad="8"/>
@@
 <via x="11.43" y="12.954" extent="1-16" drill="0.35"/>
 <via x="39.497" y="30.734" extent="1-16" drill="0.35"/>
+<contactref element="OX1" pad="6"/>
+<contactref element="OX1" pad="5"/>
+<contactref element="OX1" pad="2"/>
+<contactref element="OX1" pad="4"/>
 </signal>
 <signal name="N$1">
@@
 <contactref element="C24" pad="1"/>
 <wire x1="42.13225" y1="68.326" x2="43.65625" y2="69.85" width="0.254" layer="1"/>
-<wire x1="42.13225" y1="68.326" x2="40.64" y2="68.326" width="0.254" layer="1"/>
-<wire x1="39.116" y1="69.85" x2="40.64" y2="68.326" width="0.254" layer="1"/>
+<wire x1="42.13225" y1="68.326" x2="40.132" y2="68.326" width="0.254" layer="1"/>
+<wire x1="39.116" y1="69.342" x2="40.132" y2="68.326" width="0.254" layer="1"/>
 <wire x1="43.65625" y1="69.85" x2="45.958" y2="69.85" width="0.3048" layer="1"/>
 <wire x1="45.958" y1="69.85" x2="46.228" y2="70.27" width="0.3048" layer="1"/>
@@
 <wire x1="46.974" y1="69.374" x2="50.8" y2="69.474" width="0.3048" layer="1"/>
 <contactref element="OX1" pad="3"/>
-<wire x1="39.116" y1="69.85" x2="38.862" y2="69.85" width="0.254" layer="1"/>
-<wire x1="38.862" y1="69.85" x2="37.846" y2="70.866" width="0.254" layer="1"/>
+<wire x1="39.116" y1="69.342" x2="39.116" y2="69.596" width="0.254" layer="16"/>
+<wire x1="39.116" y1="69.596" x2="37.846" y2="70.866" width="0.254" layer="16"/>
 </signal>
 <signal name="N$29">
@@
 <contactref element="U$7" pad="1"/>
 <contactref element="K2" pad="5"/>
-<wire x1="34.6075" y1="69.37375" x2="34.6075" y2="60.80125" width="0.254" layer="1"/>
-<wire x1="34.13125" y1="69.85" x2="34.6075" y2="69.37375" width="0.254" layer="1"/>
+<wire x1="34.6075" y1="69.342" x2="34.6075" y2="60.80125" width="0.254" layer="1"/>
 <wire x1="34.6075" y1="60.80125" x2="34.753" y2="60.645" width="0.254" layer="1"/>
-<wire x1="34.13125" y1="69.85" x2="34.036" y2="69.85" width="0.254" layer="1"/>
+<wire x1="34.6075" y1="69.342" x2="34.036" y2="69.342" width="0.254" layer="1"/>
 <contactref element="OX1" pad="1"/>
-<wire x1="34.036" y1="69.85" x2="33.782" y2="69.85" width="0.254" layer="1"/>
-<wire x1="33.782" y1="69.85" x2="32.766" y2="70.866" width="0.254" layer="1"/>
+<wire x1="34.036" y1="69.342" x2="34.036" y2="69.596" width="0.254" layer="16"/>
+<wire x1="34.036" y1="69.596" x2="32.766" y2="70.866" width="0.254" layer="16"/>
 </signal>
 <signal name="RELAIS">

Commit message: Beauty Fixes
Routing:
- net GND: track 52.2 -> 31.0 mm, vias 226 -> 227
Other:
- board text added: "input switch board"
Changed lines of the file:
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@@
 <drawing>
 <settings>
-<setting alwaysvectorfont="no"/>
+<setting alwaysvectorfont="yes"/>
 <setting verticaltext="up"/>
 </settings>
@@
 <layer number="25" name="tNames" color="7" fill="1" visible="yes" active="yes"/>
 <layer number="26" name="bNames" color="7" fill="1" visible="yes" active="yes"/>
-<layer number="27" name="tValues" color="7" fill="1" visible="yes" active="yes"/>
-<layer number="28" name="bValues" color="7" fill="1" visible="yes" active="yes"/>
+<layer number="27" name="tValues" color="7" fill="1" visible="no" active="yes"/>
+<layer number="28" name="bValues" color="7" fill="1" visible="no" active="yes"/>
 <layer number="29" name="tStop" color="7" fill="3" visible="no" active="yes"/>
 <layer number="30" name="bStop" color="7" fill="6" visible="no" active="yes"/>
@@
 <layer number="43" name="vRestrict" color="2" fill="10" visible="no" active="yes"/>
 <layer number="44" name="Drills" color="7" fill="1" visible="no" active="yes"/>
-<layer number="45" name="Holes" color="7" fill="1" visible="yes" active="yes"/>
+<layer number="45" name="Holes" color="7" fill="1" visible="no" active="yes"/>
 <layer number="46" name="Milling" color="3" fill="1" visible="no" active="yes"/>
 <layer number="47" name="Measures" color="7" fill="1" visible="no" active="yes"/>
@@
 <wire x1="0" y1="5.08" x2="5.08" y2="0" width="0" layer="20" curve="100"/>
 <text x="81.661" y="53.086" size="12.7" layer="26" font="vector" rot="MR0">mb'AMP2</text>
-<text x="98.552" y="48.387" size="1.6764" layer="26" rot="MR0">maker4makers.de</text>
-<text x="98.425" y="51.943" size="1.6764" layer="26" rot="MR0">@mb'2021</text>
+<text x="67.818" y="2.921" size="1.6764" layer="26" rot="MR0">maker4makers.de</text>
+<text x="63.881" y="5.207" size="1.6764" layer="26" rot="MR0">@mb'2021</text>
 <wire x1="-4.064" y1="51.054" x2="-4.064" y2="48.514" width="0.1524" layer="48"/>
 <wire x1="-4.064" y1="48.514" x2="-4.064" y2="46.736" width="0.1524" layer="48"/>
@@
 <wire x1="55.118" y1="24.13" x2="55.118" y2="14.732" width="0.4064" layer="25"/>
 <text x="54.61" y="14.986" size="1.778" layer="25" rot="R90">red</text>
-<text x="98.552" y="55.372" size="1.778" layer="26" rot="MR0">Version: 0.1</text>
+<text x="65.024" y="7.874" size="1.778" layer="26" rot="MR0">Version: 0.1</text>
+<text x="81.661" y="38.862" size="5.842" layer="26" font="vector" rot="MR0">input switch board</text>
 </plain>
 <attributes>
@@
 <contactref element="C26" pad="2"/>
 <contactref element="D3" pad="A"/>
-<wire x1="47.3075" y1="54.45125" x2="47.345" y2="54.462" width="0.254" layer="1"/>
-<wire x1="69.05625" y1="45.72" x2="69.05625" y2="52.22875" width="0.254" layer="1"/>
-<wire x1="69.05625" y1="52.22875" x2="69.024" y2="52.324" width="0.254" layer="1"/>
-<wire x1="27.14625" y1="56.03875" x2="27.153" y2="56.195" width="0.254" layer="1"/>
+<wire x1="69.024" y1="52.324" x2="69.05625" y2="52.22875" width="0.254" layer="1"/>
 <wire x1="8.1915" y1="60.67425" x2="12.6506125" y2="60.67425" width="0.254" layer="1"/>
 <wire x1="12.6506125" y1="60.67425" x2="15.576" y2="59.567" width="0.254" layer="1"/>
 <wire x1="8.1915" y1="60.67425" x2="6.604" y2="61.468" width="0.254" layer="1"/>
-<wire x1="6.604" y1="66.548" x2="6.604" y2="65.81775" width="0.254" layer="1"/>
-<wire x1="41.90890625" y1="74.13734375" x2="41.776" y2="73.842" width="0.254" layer="1"/>
-<wire x1="30.95625" y1="73.9775" x2="15.24" y2="73.9775" width="0.254" layer="1"/>
 <wire x1="31.376" y1="73.842" x2="31.029134375" y2="73.842" width="0.254" layer="1"/>
 <wire x1="31.029134375" y1="73.842" x2="30.95625" y2="73.9775" width="0.254" layer="1"/>
@@
 <via x="10.922" y="42.672" extent="1-16" drill="0.35"/>
 <via x="21.082" y="40.894" extent="1-16" drill="0.35"/>
-<wire x1="27.1485" y1="50.326" x2="26.67" y2="50.698" width="0.254" layer="1"/>
-<wire x1="30.48" y1="50.698" x2="29.718" y2="50.326" width="0.254" layer="1"/>
 <via x="24.892" y="51.562" extent="1-16" drill="0.35"/>
 <via x="32.258" y="50.292" extent="1-16" drill="0.35"/>
@@
 <wire x1="29.806" y1="23.876" x2="30.2625" y2="24.13" width="0.254" layer="1"/>
 <wire x1="30.2625" y1="24.13" x2="34.036" y2="24.13" width="0.254" layer="1"/>
-<wire x1="41.90890625" y1="74.13734375" x2="41.75125" y2="74.295" width="0.3048" layer="1"/>
 <contactref element="Q4" pad="2"/>
 <contactref element="U$1" pad="21"/>
@@
 <contactref element="U$1" pad="1"/>
 <contactref element="C21" pad="2"/>
-<wire x1="6.6675" y1="41.275" x2="6.604" y2="41.148" width="0.254" layer="1"/>
 <via x="71.374" y="44.196" extent="1-16" drill="0.35"/>
 <via x="69.088" y="44.45" extent="1-16" drill="0.35"/>
@@
 <contactref element="OX1" pad="2"/>
 <contactref element="OX1" pad="4"/>
+<via x="68.834" y="48.26" extent="1-16" drill="0.35"/>
+<wire x1="69.05625" y1="52.22875" x2="69.05625" y2="48.48225" width="0.254" layer="1"/>
+<wire x1="69.05625" y1="48.48225" x2="68.834" y2="48.26" width="0.254" layer="1"/>
 </signal>
 <signal name="N$1">
@@
 <via x="97.536" y="50.8" extent="1-16" drill="0.35"/>
 <wire x1="84.0486" y1="40.2336" x2="91.3384" y2="40.2336" width="1.016" layer="1"/>
-<wire x1="91.3384" y1="40.2336" x2="91.44" y2="40.132" width="0.3048" layer="1"/>
 <via x="54.61" y="56.896" extent="1-16" drill="0.35"/>
 <via x="54.61" y="63.246" extent="1-16" drill="0.35"/>
@@
 <via x="47.498" y="26.416" extent="1-16" drill="0.35"/>
 <via x="48.514" y="27.432" extent="1-16" drill="0.35"/>
-<wire x1="47.9425" y1="35.2425" x2="47.983" y2="35.295" width="0.254" layer="1"/>
-<wire x1="47.9425" y1="35.2425" x2="47.98303125" y2="35.29498125" width="0.254" layer="1"/>
 <via x="46.482" y="37.084" extent="1-16" drill="0.35"/>
 <via x="47.752" y="37.084" extent="1-16" drill="0.35"/>
