File: PCB-IOBoard/AMP2-IO.brd (EAGLE design)
At the start: 100.4 x 80 mm, 89 parts, among them IC1 7404TS, IC2 R-78E6.5-0.5, IC3 REG1117, IC4 REG1117, K2 GN210S03, Q4 24.576, X3 MKDSN1,5/2-5,08

Commit message: BOM optimized... more attributes
Parts:
- R1, R2: value 4.7k -> 2.2k
- R10, R11, R9: value 47 -> 75
Changed lines of the file:
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@@
 </element>
 <element name="C1" library="rcl" library_urn="urn:adsk.eagle:library:334" package="C025_050-055X075" package3d_urn="urn:adsk.eagle:package:23636/1" value="4.7u" x="80.518" y="59.69" smashed="yes" rot="R90">
+<attribute name="MINCAP" value="2.2u -&gt;30Hz" x="80.518" y="59.69" size="1.778" layer="27" rot="R90" display="off"/>
 <attribute name="NAME" x="79.502" y="55.753" size="1.27" layer="25" ratio="10"/>
 <attribute name="POPULARITY" value="1" x="80.518" y="59.69" size="1.778" layer="27" rot="R90" display="off"/>
@@
 </element>
 <element name="C2" library="rcl" library_urn="urn:adsk.eagle:library:334" package="C025_050-055X075" package3d_urn="urn:adsk.eagle:package:23636/1" value="4.7u" x="61.214" y="59.436" smashed="yes" rot="R90">
+<attribute name="MINCAP" value="2.2u -&gt;30Hz" x="61.214" y="59.436" size="1.778" layer="27" rot="R90" display="off"/>
 <attribute name="NAME" x="59.944" y="55.499" size="1.27" layer="25" ratio="10"/>
 <attribute name="POPULARITY" value="1" x="61.214" y="59.436" size="1.778" layer="27" rot="R90" display="off"/>
 <attribute name="SPICEPREFIX" value="C" x="61.214" y="59.436" size="1.778" layer="27" rot="R90" display="off"/>
 </element>
-<element name="R1" library="rcl" library_urn="urn:adsk.eagle:library:334" package="R0603" package3d_urn="urn:adsk.eagle:package:23555/3" value="4.7k" x="86.106" y="60.96" smashed="yes" rot="R270">
+<element name="R1" library="rcl" library_urn="urn:adsk.eagle:library:334" package="R0603" package3d_urn="urn:adsk.eagle:package:23555/3" value="2.2k" x="86.106" y="60.96" smashed="yes" rot="R270">
 <attribute name="NAME" x="85.344" y="59.309" size="1.27" layer="25" rot="R270"/>
 <attribute name="POPULARITY" value="70" x="86.106" y="60.96" size="1.778" layer="27" rot="R270" display="off"/>
 <attribute name="SPICEPREFIX" value="R" x="86.106" y="60.96" size="1.778" layer="27" rot="R270" display="off"/>
 </element>
-<element name="R2" library="rcl" library_urn="urn:adsk.eagle:library:334" package="R0603" package3d_urn="urn:adsk.eagle:package:23555/3" value="4.7k" x="55.88" y="60.706" smashed="yes" rot="R270">
+<element name="R2" library="rcl" library_urn="urn:adsk.eagle:library:334" package="R0603" package3d_urn="urn:adsk.eagle:package:23555/3" value="2.2k" x="55.88" y="60.706" smashed="yes" rot="R270">
 <attribute name="NAME" x="55.372" y="58.801" size="1.27" layer="25" rot="R270"/>
 <attribute name="POPULARITY" value="70" x="55.88" y="60.706" size="1.778" layer="27" rot="R270" display="off"/>
@@
 <attribute name="VALUE" x="59.69" y="48.6219" size="0.02" layer="27" rot="R270"/>
 </element>
-<element name="R9" library="rcl" library_urn="urn:adsk.eagle:library:334" package="R0603" package3d_urn="urn:adsk.eagle:package:23555/3" value="47" x="67.31" y="26.924" smashed="yes" rot="R90">
+<element name="R9" library="rcl" library_urn="urn:adsk.eagle:library:334" package="R0603" package3d_urn="urn:adsk.eagle:package:23555/3" value="75" x="67.31" y="26.924" smashed="yes" rot="R90">
 <attribute name="POPULARITY" value="70" x="67.31" y="26.924" size="1.778" layer="27" rot="R90" display="off"/>
 <attribute name="SPICEPREFIX" value="R" x="67.31" y="26.924" size="1.778" layer="27" rot="R90" display="off"/>
 <attribute name="VALUE" x="67.818" y="29.083" size="1.27" layer="27" rot="R90"/>
 </element>
-<element name="R10" library="rcl" library_urn="urn:adsk.eagle:library:334" package="R0603" package3d_urn="urn:adsk.eagle:package:23555/3" value="47" x="69.85" y="26.924" smashed="yes" rot="R90">
+<element name="R10" library="rcl" library_urn="urn:adsk.eagle:library:334" package="R0603" package3d_urn="urn:adsk.eagle:package:23555/3" value="75" x="69.85" y="26.924" smashed="yes" rot="R90">
 <attribute name="POPULARITY" value="70" x="69.85" y="26.924" size="1.778" layer="27" rot="R90" display="off"/>
 <attribute name="SPICEPREFIX" value="R" x="69.85" y="26.924" size="1.778" layer="27" rot="R90" display="off"/>
 <attribute name="VALUE" x="70.104" y="29.083" size="1.27" layer="27" rot="R90"/>
 </element>
-<element name="R11" library="rcl" library_urn="urn:adsk.eagle:library:334" package="R0603" package3d_urn="urn:adsk.eagle:package:23555/3" value="47" x="72.39" y="26.924" smashed="yes" rot="R90">
+<element name="R11" library="rcl" library_urn="urn:adsk.eagle:library:334" package="R0603" package3d_urn="urn:adsk.eagle:package:23555/3" value="75" x="72.39" y="26.924" smashed="yes" rot="R90">
 <attribute name="POPULARITY" value="70" x="72.39" y="26.924" size="1.778" layer="27" rot="R90" display="off"/>
 <attribute name="SPICEPREFIX" value="R" x="72.39" y="26.924" size="1.778" layer="27" rot="R90" display="off"/>

Commit message: Quick fixes to RC1
Parts:
- moved IC2 14.1 mm to (91.7, 17.0)
- moved L1 8.89 mm to (85.1, 26.2)
- moved C4 1.52 mm to (92.2, 32.8)
Routing:
- net +7V: track 123.4 -> 143.0 mm
- net N$20: track 30.3 -> 44.7 mm
- net N$5: track 38.2 -> 30.9 mm
- added copper zone on layer 1, net N$20
- added copper zone on layer 1, net VIN2
Other:
- board text added: "Version: 1.0-RC2"
- board text removed: "Version: 0.1"

Commit message: Some fixes..
Parts:
- R1, R2: value 2.2k -> 4.7k
- R10, R11, R9: value 75 -> 47
- moved IC2 14.1 mm to (80.8, 8.13)
- moved L1 8.89 mm to (85.1, 17.3)
- moved C4 1.52 mm to (92.2, 31.2)
- renumbered SRCLOCK to SRCUNLOCK
Connections:
- net N$10 renamed AD_LRCK
- net N$11 renamed AD_DOUT
- net N$12 renamed RX_DOUT
- net N$13 renamed VREF1
- net N$14 renamed VREF2
- net N$6 renamed RX_SCK
- net N$7 renamed RX_BCK
- net N$8 renamed RX_LRCK
- net N$9 renamed AD_BCK
- removed net GND1: SV3.7, SV3.8
- net GND: now also SV3.7, SV3.8
Routing:
- net +7V: track 143.0 -> 123.4 mm
- net N$20: track 44.7 -> 30.3 mm
- net N$5: track 30.9 -> 38.2 mm
- net GND: track 30.9 -> 36.0 mm, vias 227 -> 226
- net GND1: track 2.59 -> 0.00 mm
- removed copper zone on layer 1, net N$20
- removed copper zone on layer 1, net VIN2
Other:
- board text added: "Version: 0.1"
- board text removed: "Version: 1.0-RC2"
- board text removed: "input switch board"

Commit message: Some RC1 bugs fixed.
Parts:
- added C22: 10n, rcl:C0603
- added JMP1: 0R-JUMPA, jump-0r-smd:A0R-JMP
- added R22, R23: 4.7k, rcl:R0603
- added R8: 220, rcl:R0603
- moved R11 5.36 mm to (67.1, 27.4)
- moved R9 1.85 mm to (69.1, 27.4)
- moved R10 1.37 mm to (71.1, 27.4)
- turned L3 to 90 degrees
- flipped SV4 to the bottom
Connections:
- new net N$6: JMP1.2, L3.1
- new net N$7: C22.2, R8.1
- new net N$8: K2.6, R8.2
- net +3V3: now also JMP1.1
- net A5V: now also JMP1.3
- net GND: now also R22.1, R23.1; no longer L3.1
- net N$19: now also C22.1; no longer K2.6
- net SEL_A: now also R22.2
- net SEL_B: now also R23.2
Routing:
- net +3V3: track 179.0 -> 241.4 mm
- net A5V: track 38.0 -> 64.7 mm
- net N$19: track 34.4 -> 12.9 mm
- net SCL: track 89.5 -> 107.9 mm, vias 3 -> 4
- net N$8: track 0.00 -> 16.6 mm
- net SDA: track 86.7 -> 100.7 mm, vias 3 -> 4
- net RESET: track 90.5 -> 81.8 mm, vias 1 -> 2
- net N$25: track 12.8 -> 8.18 mm
- net LRCLK: track 6.81 -> 10.9 mm, vias 0 -> 1
- net N$6: track 0.00 -> 2.93 mm
- net SRC_LOCK: track 69.8 -> 71.8 mm
- net N$7: track 0.00 -> 1.86 mm
- net GND: track 36.0 -> 34.2 mm
- net DOUT_EX1: track 64.6 -> 62.9 mm
- net SEL_A: track 43.8 -> 45.1 mm
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
Commit message: More fixes on AMP2-IO.
Parts:
- K2: value GN210S03 -> GN200S03
Connections:
- net +3V3: no longer U$2.28
- net ERROR: now also U$2.28
- net GND: now also K2.8; no longer K2.1
- net N$35: now also K2.1; no longer K2.8
Routing:
- net N$35: track 26.1 -> 30.1 mm
- net +3V3: track 241.4 -> 238.1 mm
- net ERROR: track 33.6 -> 36.6 mm
