File: PCB-IOBoard/AMP2-IO.sch (EAGLE design)
At the start: 37 parts, among them IC3 REG1117, IC4 REG1117

Commit message: Getting somewhere.
Parts:
- removed SV1: (no value), con-lsta:FE10-2
- removed SV2: (no value), con-lsta:FE08-1
- added C18, C19: 100u, rcl:CPOL-EU153CLV-0807
- added C20: 100n, rcl:C-EUC0805K
- added C21, C22: 12p, rcl:C-EUC0805K
- added Q2: 12.288, crystal:CRYSTALCTS406
- added R10, R11, R9: 47, rcl:R-EU_R0805W
- added R6, R8: 4.02k, rcl:R-EU_R0805W
- added R7: 1k, rcl:R-EU_R0805W
- added SJ1: (no value), jumper:SJ
- added SV3: (no value), con-lsta:FE08-1
- added SV4: (no value), con-lsta:FE10-2
- C3, C4: device rcl:CPOL-EU153CLV-1010 -> rcl:CPOL-EU153CLV-0807
- C5: value (none) -> 100n
- L1: device rcl:L-EUL5650M -> rcl:L-EUL4532P
- L2: device rcl:L-EUL5650M -> rcl:L-EUL4532C
- SPDIF: MOUSER (none) -> 502-PJRAN1X1U01AUX; MOUSER2 (none) -> 502-PJRAN1X1U02AUX
Connections:
- new net +5V: C18.+, IC4.VIN, SV3.3, SV3.4
- new net ADR/FAULT: SV4.1
- new net GND1: SV3.7, SV3.8
- new net LRCLK: R9.1, SV4.13
- new net MCLK: U$1.MCLK_OUT, U$3.SCKI
- new net N$20: C21.2, Q2.1, U$1.XTI
- new net N$21: R6.1, U$1.MS_SEL
- new net N$22: R7.1, U$1.SAIF
- new net N$23: R8.1, U$1.SAOF
- new net N$24: C22.2, Q2.2, U$1.XTO
- new net N$25: R11.2, U$1.SDOUT
- new net N$26: R10.2, U$1.OSCLK
- new net N$27: R9.2, U$1.OLRCK
- new net PDN: SV4.3
- new net SCL: SV4.17, U$4.SCL
- new net SCLK: R10.1, SV4.11
- new net SDA: SV4.15, U$4.SDA
- new net SDIN: R11.1, SV4.7
- new net SDOUT: SV4.9
- net +12V: now also SV3.1, SV3.2
- net +3V3: now also C19.+, C5.1, SV3.5, SV3.6, U$3.FMT0, U$3.MODE0, U$3.MODE1, U$3.PDWN
- net A5V: now also C20.1
- net AGND: now also C20.2, SJ1.1
- net GND: now also C18.-, C19.-, C21.1, C22.1, C5.2, IC4.GND, R6.2, R7.2, R8.2, SJ1.2, SV4.10, SV4.12, SV4.14, SV4.16, SV4.18, SV4.20, SV4.6, SV4.8, U$3.BYPAS, U$3.FMT1, U$3.OSR
- net SW_BCK: now also U$1.ISCLK
- net SW_SCLK: no longer U$1.ISCLK
Other:
- note added: "(MCLK)"
- note added: "Add Sys Clock 2-50MHz"
- note added: "CKSEL=0 > recover CLK used 24.576-MHz clock on the XTI pin FMT01 = H > I2S format RESET? PSCK = L > 128fs, max 6.144MHz Wenn alle Slav'n kann man umschalter sparen !"
- note added: "SlaveIn, MasterOut In i2s Out i2s 24bit 256fs"
- note removed: "CKSEL=0 > recover CLK used 24.576-MHz clock on the XTI pin FMT01 = H > I2S format RESET? PSCK = L > 128fs, max 6.144MHz"
- moved on the sheet: C1, C10, C11, C12, C13, C14, C15, C16, C17, C2, C3, C4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

Commit message: Added Ext Headers, TORX, ... not complete yet.
Parts:
- added C23: 10u, rcl:CPOL-EU153CLV-0807
- added C24: 100n, rcl:C-EUC0805K
- added C25: 4.7n, rcl:C-EUC0805K
- added D1, D2: (no value), diode:SCHOTTKY-DIODESMD
- added EXT1, EXT2: (no value), con-lsta:FE08-1
- added IC1: 7404D, 74xx-eu:7404D
- added IC2: R-78E-0.5, linear:788TV
- added L3: (no value), rcl:L-EUL4532P
- added L5: 10uH, inductors:DR125
- added SJ2: (no value), jumper:SJ
- added SV1: (no value), con-lsta:FE05-1
- added U$7: TORX135X, AMP2-ICs:TORX135X
- added X3: MKDSN1,5/2-5,08, con-phoenix-508:MKDSN1,5/2-5,08
- C18: value 100u -> 10u
- C4: value (none) -> 10u
- R3: value 0 -> 680; device rcl:R-EU_R1206W -> rcl:R-EU_R0805W
Connections:
- removed net +5V: C18.+, IC4.VIN, SV3.3, SV3.4
- new net +7V: C18.+, IC2.VO, IC4.VIN, L1.1
- new net BCLK_EX1: EXT1.6, U$5G$1.Y2
- new net BCLK_EX2: EXT2.6, U$5G$1.Y3
- new net DOUT_EX1: EXT1.4, U$6G$1.Y2
- new net DOUT_EX2: EXT2.4, U$6G$1.Y3
- new net ERNIE: D1.A, L5.2
- new net GP6: EXT1.2, U$4.GP6
- new net GP7: EXT2.2, U$4.GP7
- new net HORST: L5.1, X3-2.KL
- new net LRCK_EX1: EXT1.5, U$6G$1.X2
- new net LRCK_EX2: EXT2.5, U$6G$1.X3
- new net N$28: C24.1, L3.2, U$7.VCC
- new net N$29: IC1A.I, IC1B.O
- new net N$30: C23.+, D1.C, D2.C, IC2.VI
- new net N$31: C25.1, R3.1, SPDIF.2
- new net N$32: C25.2, IC1B.I
- new net SCLK_EX1: EXT1.7, U$5G$1.X2
- new net SCLK_EX2: EXT2.7, U$5G$1.X3
- net +12V: now also D2.A; no longer L1.1
- net +3V3: now also EXT1.8, EXT2.8, IC1P.VCC, U$4.VDD; no longer SV3.5, SV3.6
- net AGND: now also C24.2, IC1C.I, IC1D.I, IC1E.I, IC1F.I, IC1P.GND, L3.1, SJ2.1, U$7.GND@2
- net GND: now also C23.-, EXT1.1, EXT1.3, EXT2.1, EXT2.3, IC2.GND, SJ2.2, SV1.1, U$4.GND, X3-1.KL; no longer R3.1
- net N$19: now also U$7.OUT
- net SCL: now also SV1.2
- net SDA: now also SV1.3
Other:
- note added: "Power Options: * Header provides 12V+ (can be 9-24V fom AMP) * External 9-24V IC2 does StepDown to 7V and supplies the 2 linear regulators."
- moved on the sheet: R3, SPDIF

Commit message: Autorouted and Manual Layout
Parts:
- added C26, C27: 100n, rcl:C-EUC0805K
- added D3: MBR0520LT, diode:MBR0520LT
- added K2: GN210S03, relay:GN210S03
Connections:
- new net N$33: K2T.S, U$7.OUT
- new net N$34: IC1A.O, K2T.O
- new net N$35: D3.C, IC1C.O, IC1D.O, IC1E.O, IC1F.O, K2R.+
- new net RELAIS: IC1C.I, IC1D.I, IC1E.I, IC1F.I, U$4.GP2
- net +3V3: now also C26.1, C27.1, U$1.VD, U$1.VL
- net AGND: no longer IC1C.I, IC1D.I, IC1E.I, IC1F.I, IC1P.GND
- net GND: now also C26.2, C27.2, D3.A, IC1P.GND, K2R.-, U$1.GND, U$1.GND2
- net N$19: now also K2T.P; no longer U$7.OUT
Other:
- moved on the sheet: IC1C, IC1D, IC1E, IC1F

Commit message: Routed.
Parts:
- added FS1, FS2, POWER, RX_ERROR, SRCUNLOCK: (no value), led:LEDCHIPLED_0805
- added R12, R13, R14, R15, R16, R20: 1k, rcl:R-EU_R0805W
- added R17: 47k, rcl:R-EU_R0805W
- added R18: 2.2k, rcl:R-EU_R0805W
- added R19: 4.02k, rcl:R-EU_R0805W
- added R21: open, rcl:R-EU_R0805W
- added SRC_BYPASS: (no value), jumper:JP1E
- C25: value 4.7n -> 10n
- IC2: value R-78E-0.5 -> R-78E9.0-0.5
- R3: value 680 -> 75
- R8: value 4.02k -> 8.04k
Connections:
- removed net PDN: SV4.3
- new net ERROR: R15.2, U$2.ERROR, U$4.GP5
- new net FSOUT0: R14.2, U$2.FSOUT0, U$4.GP4
- new net FSOUT1: R13.2, U$2.FSOUT1, U$4.GP3
- new net N$36: POWER.A, R12.1
- new net N$37: FS1.A, R13.1
- new net N$38: FS2.A, R14.1
- new net N$39: R15.1, RX_ERROR.A
- new net N$40: R16.1, SRCUNLOCK.A
- new net N$41: R19.2, SRC_BYPASS.1, U$1.BYPASS
- new net N$42: R20.1, R21.2, U$4.ADDR
- new net SRC_UNLOCK: R16.2, U$1.SRC_UNLOCK, U$4.GP6
- net +3V3: now also R12.2, R21.1, SRC_BYPASS.2
- net AGND: no longer C24.2, L3.1, R3.2, SPDIF.1, U$7.GND@2
- net GND: now also C24.2, FS1.C, FS2.C, IC1C.I, L3.1, POWER.C, R18.1, R19.1, R20.2, R3.2, RX_ERROR.C, SPDIF.1, SRCUNLOCK.C, U$1.TDM_IN, U$7.GND@2
- net GP6: no longer U$4.GP6
- net GP7: now also U$4.GP2; no longer U$4.GP7
- net N$29: now also R17.2, R18.2
- net N$32: now also R17.1
- net N$35: no longer IC1C.O
- net RELAIS: now also U$4.GP7; no longer IC1C.I, U$4.GP2
- net RESET: now also SV4.3, U$1.RST
Other:
- note added: "4.02k for 24bit out"
- note added: "8.04k for 32bit out"
- note added: "Bypass Switch"
- note added: "CONV"
- note added: "EXT2"
- note added: "INPUT SEL"
- note added: "NC"
- note added: "PDN"
- note added: "SPDIF"
- note added: "adr=0x40 (8bit)"
- note added: "https://www.conrad.de/de/p/cliff-lwl-steckverbinder-fcr684205r-toslink-empfaenger-457611.html"
- note added: "ohne ext CLK, kein FS"
- moved on the sheet: C21, C22, EXT1, EXT2, IC1A, IC1C, Q2, R6, R7, R8, SV1, SV4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

Commit message: Switched to SRC4192
Parts:
- removed C22: 12p, rcl:C-EUC0805K
- removed Q2: 12.288, crystal:CRYSTALCTS406
- removed R7: 1k, rcl:R-EU_R0805W
- removed R8: 8.04k, rcl:R-EU_R0805W
- added Q4: 12.288, crystal-geyer_V1_0:KXO-TCXO-CMOS-82
- C18, C19, C23, C3, C4: device rcl:CPOL-EU153CLV-0807 -> rcl:CPOL-EUCT6032
- C21: value 12p -> 100n
- C25: value 10n -> 100n
- R6: value 4.02k -> 1k
- U$1: value CS8421 -> SRC4192; device AMP2-ICs:CS8421 -> AMP2-ICs:SRC4192
- renumbered SRCUNLOCK to SRCLOCK
Connections:
- net HORST renamed VIN
- net N$30 renamed VIN2
- removed net N$20: C21.2, Q2.1, U$1.XTI
- removed net N$21: R6.1, U$1.MS_SEL
- removed net N$22: R7.1, U$1.SAIF
- removed net N$23: R8.1, U$1.SAOF
- removed net N$24: C22.2, Q2.2, U$1.XTO
- removed net SRC_UNLOCK: R16.2, U$1.SRC_UNLOCK, U$4.GP6
- new net SRC_LOCK: R16.2, U$1./RDY, U$1.MUTE, U$4.GP6
- net +3V3: now also C21.1, Q4.VDD, U$1.IFMT0, U$1.MODE0, U$1.OFMT0, U$1.VDD, U$1.VIO; no longer U$1.VD, U$1.VL
- net AGND: no longer C14.2, C15.2, C16.1, C17.1, U$2.AGND
- net GND: now also C14.2, C15.2, C16.1, C17.1, C21.2, Q4.GND, U$1.GND@21, U$1.GND@8, U$1.IFMT1, U$1.IFMT2, U$1.LGRP, U$1.MODE1, U$1.MODE2, U$1.OFMT1, U$1.OWL0, U$1.OWL1, U$1.TDMI, U$2.AGND; no longer C21.1, C22.1, R7.2, R8.2, U$1.GND, U$1.GND2, U$1.TDM_IN
- net MCLK: now also Q4.OUT, U$1.RCKI; no longer U$1.MCLK_OUT
- net N$26: now also U$1.BCKO; no longer U$1.OSCLK
- net N$27: now also U$1.LRCKO; no longer U$1.OLRCK
- net N$41: now also U$1.BYPAS; no longer U$1.BYPASS
- net RELAIS: now also R6.1
- net RESET: now also U$1./RST; no longer U$1.RST
- net SW_BCK: now also U$1.BCKI; no longer U$1.ISCLK
- net SW_LRCK: now also U$1.LRCKI; no longer U$1.ILRCK
Other:
- note added: "nc"
- note added: "output master 96kHz"
- note removed: "4.02k for 24bit out"
- note removed: "8.04k for 32bit out"
- moved on the sheet: C21, R19, R6, SRC_BYPASS

Commit message: 603 packs and some other stuff. Changed MCLK to 24.576 needed by DIR9001 for FS detection.
Parts:
- added OX1: TORX173, toshiba:TORX173
- C10: MOUSER (none) -> 81-GCM32DL81A106KA7L
- C11, C13, C15, C16, C17, C20, C21, C24, C25, C26, C27, C5, C6, C7: device rcl:C-EUC0805K -> rcl:C-EUC0603
- C19: value 100u -> 10u
- C23: MOUSER (none) -> 80-T491C106K25AT7280
- C3: value (none) -> 10u
- D3: MOUSER (none) -> 863-MBR130T3G
- IC1: MOUSER (none) -> 595-SN74HC04DRG4
- IC2: MOUSER (none) -> 919-R-786.5-0.5
- IC3: MOUSER (none) -> 863-LM1117MPX-50NOPB
- IC4: MOUSER (none) -> 863-LM1117MPX-33NOPB
- L1, L3: value (none) -> 220uH; device rcl:L-EUL4532P -> rcl:L-EUL4532C; MOUSER (none) -> 710-7447669220
- L2: value (none) -> 220uH; MOUSER (none) -> 710-7447669220
- L5: MOUSER (none) -> 710-7447669220
- Q4: value 12.288 -> 24.576; MOUSER (none) -> 998-1001AI2024.5760T
- R1, R10, R11, R17, R18, R2, R21, R3, R5, R9: device rcl:R-EU_R0805W -> rcl:R-EU_R0603
- R12, R13, R14, R15, R16, R20, R4, R6: value 1k -> 2.2k; device rcl:R-EU_R0805W -> rcl:R-EU_R0603
- R19: value 4.02k -> 2.2k; device rcl:R-EU_R0805W -> rcl:R-EU_R0603
- U$1: MOUSER (none) -> 595-SRC4192IDB
- U$2: MOUSER (none) -> 595-DIR9001PW
- U$3: MOUSER (none) -> 595-PCM1802
- U$4: MOUSER (none) -> 579-MCP23009T-E/SS
- U$6: MOUSER (none) -> 595-SN74LV4052APWR
- U$7: MOUSER (none) -> 757-TORX1355VF
Connections:
- net +3V3: now also U$1.MODE1, U$2.CKSEL
- net GND: no longer U$1.MODE1, U$2.CKSEL
- net MCLK: now also U$2.XTI
- net N$28: now also OX1.VCC
- net N$33: now also OX1.OUT

Commit message: Changed switching chipies to SN74CBT3253.
Parts:
- removed L5: 10uH, inductors:DR125
- U$5: value CD4052B -> SN74CBT3253; device AMP2-ICs:CD4052B -> AMP2-ICs:SN74CBT3253
- U$6: value CD4052B -> SN74CBT3253; device AMP2-ICs:CD4052B -> AMP2-ICs:SN74CBT3253; MOUSER 595-SN74LV4052APWR -> (none)
Connections:
- removed net VIN: L5.1, X3-2.KL
- net +3V3: now also U$5G$1.VCC, U$6G$1.VCC; no longer U$5G$2.VCC, U$6G$2.VCC
- net BCLK_EX1: now also U$5G$2.2B3; no longer U$5G$1.Y2
- net BCLK_EX2: now also U$5G$2.2B4; no longer U$5G$1.Y3
- net DOUT_EX1: now also U$6G$2.2B3; no longer U$6G$1.Y2
- net DOUT_EX2: now also U$6G$2.2B4; no longer U$6G$1.Y3
- net ERNIE: now also X3-2.KL; no longer L5.2
- net GND: now also U$5G$1.GND, U$5G$2./1OE, U$5G$2./2OE, U$6G$1.GND, U$6G$2./1OE, U$6G$2./2OE; no longer U$5G$1.INH, U$5G$2.GND, U$5G$2.VEE, U$6G$1.INH, U$6G$2.GND, U$6G$2.VEE
- net LRCK_EX1: now also U$6G$2.1B3; no longer U$6G$1.X2
- net LRCK_EX2: now also U$6G$2.1B4; no longer U$6G$1.X3
- net N$10: now also U$6G$2.1B2; no longer U$6G$1.X1
- net N$11: now also U$6G$2.2B2; no longer U$6G$1.Y1
- net N$12: now also U$6G$2.2B1; no longer U$6G$1.Y0
- net N$6: now also U$5G$2.1B1; no longer U$5G$1.X0
- net N$7: now also U$5G$2.2B1; no longer U$5G$1.Y0
- net N$8: now also U$6G$2.1B1; no longer U$6G$1.X0
- net N$9: now also U$5G$2.2B2; no longer U$5G$1.Y1
- net SCLK_EX1: now also U$5G$2.1B3; no longer U$5G$1.X2
- net SCLK_EX2: now also U$5G$2.1B4; no longer U$5G$1.X3
- net SEL_A: now also U$5G$2.S0, U$6G$2.S0; no longer U$5G$1.A, U$6G$1.A
- net SEL_B: now also U$5G$2.S1, U$6G$2.S1; no longer U$5G$1.B, U$6G$1.B
- net SW_BCK: now also U$5G$2.2A; no longer U$5G$1.Y
- net SW_DOUT: now also U$6G$2.2A; no longer U$6G$1.Y
- net SW_LRCK: now also U$6G$2.1A; no longer U$6G$1.X
- net SW_SCLK: now also U$5G$2.1A; no longer U$5G$1.X
Other:
- note added: "FROM TAS58xx"
- note added: "screw terminal"
- moved on the sheet: C23, D1, D2, IC2, SV3, X3-1, X3-2
