File: PCB-Eagle/AMP2.brd (EAGLE design)
At the start: 100 x 80 mm, 19 parts, among them IC1 LD117AS33TR, X1 MKDSN1,5/2-5,08, X2 MKDSN1,5/2-5,08, X3 MKDSN1,5/2-5,08

Commit message: longer todo list :(
Parts:
- added SV1: (no value), con-lsta:FE05-1
- added SV2: (no value), con-lsta:FE08-2
- moved X3 41.7 mm to (48.3, 74.9), turned to 0 degrees
- moved IC1 33.1 mm to (30.5, 38.1)
- moved C8 5.08 mm to (55.9, 72.4)
- moved C5 5.08 mm to (25.4, 72.4)
- moved C6 5.08 mm to (40.6, 72.4)
- moved C7 5.08 mm to (71.1, 72.4)
- moved R5 3.81 mm to (47.0, 34.3), turned to 270 degrees
- moved R6 3.81 mm to (49.5, 34.3), turned to 270 degrees
Connections:
- new net SCL: SV1.4, U$1.11
- new net SDA: SV1.3, U$1.10
- net GND: now also SV1.5

Commit message: Removed Pi header, added power filter.
Parts:
- removed X1, X2: MKDSN1,5/2-5,08, con-phoenix-508:MKDSN1,5/2-5,08
- added C10, C9: 1u, rcl:C1206
- added C11, C13, C16: .1u, rcl:C1206
- added C12: 10u, rcl:C1210
- added C14, C15, C17, C18, C19, C21: 220u, rcl:150CLZ-1010
- added D1: (no value), diode:SMC
- added H1, H2, H3, H4: MOUNT-HOLE3.2, holes:3,2
- added H5, H6: MOUNT-HOLE3.2, holes:2,8
- added IC2: R-78E-0.5, linear:TO220V
- added L5: 10uH, inductors:DR125
- added LED1: (no value), led:1206
- added OUT-L, OUT-R: MKDSN1,5/2-5,08, con-phoenix-508:MKDSN1,5/2-5,08
- added R1: 220, rcl:R1206
- added SJ1, SJ2: (no value), jumper:SJ
- added SV3: (no value), con-lsta:FE08
- C5, C6, C7, C8: value 2.2n -> 680n
- R5: value (none) -> 4.7k
- R6: value (none) -> 10k
- moved X3 68.4 mm to (30.5, 8.89)
- moved SV2 35.4 mm to (67.3, 24.1), turned to 180 degrees
- moved IC1 13.0 mm to (27.9, 25.4), turned to 0 degrees
- moved R6 9.92 mm to (43.2, 26.7), turned to 180 degrees
- moved R5 6.35 mm to (43.2, 29.2), turned to 180 degrees
- moved C1 4.58 mm to (38.1, 48.3)
- moved SV1 3.81 mm to (49.5, 22.9)
- moved U$1 2.84 mm to (49.5, 39.4)
- moved C3 2.54 mm to (62.2, 48.3)
- moved C8 2.54 mm to (58.4, 72.4)
- moved L4 2.54 mm to (58.4, 61.0)
- moved C7 2.54 mm to (73.7, 72.4)
- moved L3 2.54 mm to (73.7, 61.0)
- moved C4 1.27 mm to (53.3, 50.8)
- moved C5 1.27 mm to (26.7, 72.4)
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Connections:
- new net +5V: IC1.3, IC2.3, SJ2.1, SV3.3, SV3.4
- new net ADR/FAULT: R5.1, SV1.1, U$1.3
- new net ERNIE: D1.A, L5.2
- new net HORST: L5.1, X3.2
- new net LRCLK: SV2.9, U$1.6
- new net N$15: C10.2, U$1.4
- new net N$16: C9.2, U$1.13
- new net N$19: SJ2.2, SV2.1
- new net PDN: R6.1, SJ1.1, SV1.2, U$1.12
- new net SCLK: SV2.7, U$1.7
- new net SDIN: SV2.3, U$1.8
- new net SDOUT: SV2.5, U$1.9
- net +12V: now also C13.2, C14.+, C15.+, C16.2, C17.+, C18.+, C19.+, C21.+, D1.C, IC2.1, SV3.1, SV3.2; no longer IC1.3, X3.2
- net +3V3: now also C11.2, C12.2, LED1.C, SV3.5, SV3.6
- net GND: now also C10.1, C11.1, C12.1, C13.1, C14.-, C15.-, C16.1, C17.-, C18.-, C19.-, C21.-, C9.1, IC2.2, R1.1, SV2.10, SV2.12, SV2.14, SV2.16, SV2.2, SV2.4, SV2.6, SV2.8, SV3.7, SV3.8; no longer U$1.9
- net N$1: now also OUT-L.1; no longer X1.1
- net N$10: now also OUT-L.2; no longer X1.2
- net N$11: now also OUT-R.2; no longer X2.2
- net N$12: now also OUT-R.1; no longer X2.1
- net N$13: now also LED1.A, R1.2; no longer R6.1, U$1.12
- net N$14: now also SJ1.2, SV2.15; no longer R5.1, U$1.3
- net SCL: now also SV2.13
- net SDA: now also SV2.11
Routing:
- net +5V: track 0.00 -> 72.2 mm
- net +3V3: track 0.00 -> 63.9 mm, vias 0 -> 1
- net SDIN: track 0.00 -> 33.1 mm
- net SDA: track 0.00 -> 31.2 mm, vias 0 -> 1
- net SDOUT: track 0.00 -> 31.0 mm, vias 0 -> 1
- net SCLK: track 0.00 -> 29.3 mm
- net N$4: track 0.00 -> 28.0 mm
- net LRCLK: track 0.00 -> 27.7 mm
- net N$2: track 0.00 -> 27.4 mm
- net SCL: track 0.00 -> 26.4 mm, vias 0 -> 1
- net +12V: track 0.00 -> 26.4 mm, vias 0 -> 43
- net PDN: track 0.00 -> 22.4 mm, vias 0 -> 2
- net ADR/FAULT: track 0.00 -> 17.5 mm, vias 0 -> 1
- net N$5: track 0.00 -> 17.1 mm
- net N$3: track 0.00 -> 16.4 mm
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- added copper zone on layer 1, net +12V
- added copper zone on layer 16, net +12V
- added copper zone on layer 1, net ERNIE
- added copper zone on layer 16, net GND
- added copper zone on layer 1, net HORST
Other:
- board size 100 x 80 mm -> 100.4 x 80 mm
- board text added: "(5V)"
- board text added: "+"
- board text added: "+12V"
- board text added: "+3.3V"
- board text added: "+5V"
- board text added: "-"
- board text added: "6-26V"
- board text added: "@mb'2020"
- board text added: "ADR"
- board text added: "FAULT"
- board text added: "GND"
- board text added: "LRCLK"
- board text added: "PDN"
- board text added: "R6"
- board text added: "Raspberry Zero (W)"
- board text added: "SCL"
- board text added: "SCLK"
- board text added: "SDA"
- board text added: "SDIN"
- board text added: "SDOUT"
- board text added: "maker4makers.de"
- board text added: "mb'AMP2"
- board text added: "red"

Commit message: rev2..
Parts:
- removed H5, H6: MOUNT-HOLE3.2, holes:2,8
- removed SJ1: (no value), jumper:SJ
- removed SV1: (no value), con-lsta:FE05-1
- removed SV2: (no value), con-lsta:FE08-2
- added SV4: (no value), con-lsta:FE10-2
- moved SJ2 24.2 mm to (52.1, 17.8), turned to 0 degrees
- moved C10 10.3 mm to (43.2, 23.7), turned to 0 degrees
- moved SV3 7.97 mm to (27.4, 18.0), turned to 0 degrees
- moved IC1 5.08 mm to (22.9, 25.4), turned to 270 degrees
- moved C12 1.27 mm to (36.8, 25.4), turned to 270 degrees
- moved OUT-L 1.27 mm to (34.3, 71.1)
- moved OUT-R 1.27 mm to (66.0, 71.1)
- moved X3 0.13 mm to (30.5, 9.02)
Connections:
- removed net N$19: SJ2.2, SV2.1
- net ADR/FAULT: now also SV4.1; no longer SV1.1
- net GND: now also SV4.10, SV4.12, SV4.14, SV4.16, SV4.18, SV4.20, SV4.6, SV4.8; no longer SV1.5, SV2.10, SV2.12, SV2.14, SV2.16, SV2.2, SV2.4, SV2.6, SV2.8
- net LRCLK: now also SV4.13; no longer SV2.9
- net N$14: now also SJ2.2, SV4.5; no longer SJ1.2, SV2.15
- net PDN: now also SV4.3; no longer SJ1.1, SV1.2
- net SCL: now also SV4.17; no longer SV1.4, SV2.13
- net SCLK: now also SV4.11; no longer SV2.7
- net SDA: now also SV4.15; no longer SV1.3, SV2.11
- net SDIN: now also SV4.7; no longer SV2.3
- net SDOUT: now also SV4.9; no longer SV2.5
Routing:
- net +5V: track 72.2 -> 46.8 mm
- net +12V: track 26.4 -> 2.88 mm
- net LRCLK: track 27.7 -> 39.9 mm
- net SCL: track 26.4 -> 38.6 mm, vias 1 -> 0
- net PDN: track 22.4 -> 33.1 mm
- net SDOUT: track 31.0 -> 39.0 mm, vias 1 -> 0
- net ADR/FAULT: track 17.5 -> 24.8 mm
- net N$15: track 12.0 -> 18.4 mm, vias 0 -> 2
- net SDA: track 31.2 -> 37.1 mm, vias 1 -> 0
- net +3V3: track 63.9 -> 58.6 mm
- net HORST: track 0.00 -> 3.79 mm, vias 0 -> 1
- net N$11: track 10.8 -> 14.1 mm, vias 0 -> 1
- net N$10: track 10.8 -> 14.1 mm, vias 0 -> 1
- net N$1: track 10.7 -> 14.0 mm, vias 0 -> 1
- net N$12: track 10.7 -> 14.0 mm, vias 0 -> 1
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Other:
- outline, holes or cut-outs redrawn
- board text added: "1"
- board text added: "freedsp header"

Commit message: v02
Parts:
- added FAULT: (no value), led:1206
- added R2: 220, rcl:R1206
Connections:
- new net N$17: FAULT.C, R2.1
- net +3V3: now also R2.2
- net ADR/FAULT: now also FAULT.A
Routing:
- net ADR/FAULT: track 24.8 -> 40.1 mm
- net +3V3: track 58.6 -> 65.5 mm
- net N$17: track 0.00 -> 2.24 mm
Other:
- outline, holes or cut-outs redrawn
- board text added: "120k 0x5e"
- board text added: "15k 0x5a"
- board text added: "4.7k 0x58"
- board text added: "47k 0x5c"
- board text added: "< 8x GND"
- board text added: "A"
- board text added: "B"
- board text added: "R5 ADR"
- board text added: "power2header >"

Commit message: Getting somewhere.
Other:
- board text removed: "Raspberry Zero (W)"
Changed lines of the file:
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@@
 <text x="60.198" y="15.367" size="1.016" layer="25" rot="R90">PDN</text>
 <text x="57.658" y="13.97" size="1.016" layer="25" rot="R90">FAULT</text>
-<text x="41.91" y="11.43" size="1.016" layer="25" font="vector">Raspberry Zero (W)</text>
 <circle x="45.339" y="35.306" radius="0.283978125" width="0.1524" layer="25"/>
 <text x="25.654" y="75.057" size="2.54" layer="25">+</text>

Commit message: Added Ext Headers, TORX, ... not complete yet.
Changed lines of the file:
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@@
 <grid distance="50" unitdist="mil" unit="mil" style="lines" multiple="1" display="yes" altdistance="5" altunitdist="mil" altunit="mil"/>
 <layers>
-<layer number="1" name="Top" color="4" fill="1" visible="yes" active="yes"/>
+<layer number="1" name="Top" color="4" fill="1" visible="no" active="yes"/>
 <layer number="2" name="Route2" color="1" fill="3" visible="no" active="no"/>
 <layer number="3" name="Route3" color="4" fill="3" visible="no" active="no"/>
@@
 <layer number="14" name="Route14" color="1" fill="6" visible="no" active="no"/>
 <layer number="15" name="Route15" color="4" fill="6" visible="no" active="no"/>
-<layer number="16" name="Bottom" color="1" fill="1" visible="yes" active="yes"/>
-<layer number="17" name="Pads" color="2" fill="1" visible="yes" active="yes"/>
-<layer number="18" name="Vias" color="2" fill="1" visible="yes" active="yes"/>
-<layer number="19" name="Unrouted" color="6" fill="1" visible="yes" active="yes"/>
-<layer number="20" name="Dimension" color="24" fill="1" visible="yes" active="yes"/>
-<layer number="21" name="tPlace" color="7" fill="1" visible="yes" active="yes"/>
-<layer number="22" name="bPlace" color="7" fill="1" visible="yes" active="yes"/>
-<layer number="23" name="tOrigins" color="15" fill="1" visible="yes" active="yes"/>
-<layer number="24" name="bOrigins" color="15" fill="1" visible="yes" active="yes"/>
+<layer number="16" name="Bottom" color="1" fill="1" visible="no" active="yes"/>
+<layer number="17" name="Pads" color="2" fill="1" visible="no" active="yes"/>
+<layer number="18" name="Vias" color="2" fill="1" visible="no" active="yes"/>
+<layer number="19" name="Unrouted" color="6" fill="1" visible="no" active="yes"/>
+<layer number="20" name="Dimension" color="24" fill="1" visible="no" active="yes"/>
+<layer number="21" name="tPlace" color="7" fill="1" visible="no" active="yes"/>
+<layer number="22" name="bPlace" color="7" fill="1" visible="no" active="yes"/>
+<layer number="23" name="tOrigins" color="15" fill="1" visible="no" active="yes"/>
+<layer number="24" name="bOrigins" color="15" fill="1" visible="no" active="yes"/>
 <layer number="25" name="tNames" color="7" fill="1" visible="yes" active="yes"/>
-<layer number="26" name="bNames" color="7" fill="1" visible="yes" active="yes"/>
-<layer number="27" name="tValues" color="7" fill="1" visible="yes" active="yes"/>
-<layer number="28" name="bValues" color="7" fill="1" visible="yes" active="yes"/>
+<layer number="26" name="bNames" color="7" fill="1" visible="no" active="yes"/>
+<layer number="27" name="tValues" color="7" fill="1" visible="no" active="yes"/>
+<layer number="28" name="bValues" color="7" fill="1" visible="no" active="yes"/>
 <layer number="29" name="tStop" color="7" fill="3" visible="no" active="yes"/>
 <layer number="30" name="bStop" color="7" fill="6" visible="no" active="yes"/>
@@
 <layer number="37" name="tTest" color="7" fill="1" visible="no" active="yes"/>
 <layer number="38" name="bTest" color="7" fill="1" visible="no" active="yes"/>
-<layer number="39" name="tKeepout" color="4" fill="11" visible="yes" active="yes"/>
-<layer number="40" name="bKeepout" color="1" fill="11" visible="yes" active="yes"/>
-<layer number="41" name="tRestrict" color="4" fill="10" visible="yes" active="yes"/>
-<layer number="42" name="bRestrict" color="1" fill="10" visible="yes" active="yes"/>
+<layer number="39" name="tKeepout" color="4" fill="11" visible="no" active="yes"/>
+<layer number="40" name="bKeepout" color="1" fill="11" visible="no" active="yes"/>
+<layer number="41" name="tRestrict" color="4" fill="10" visible="no" active="yes"/>
+<layer number="42" name="bRestrict" color="1" fill="10" visible="no" active="yes"/>
 <layer number="43" name="vRestrict" color="2" fill="10" visible="no" active="yes"/>
 <layer number="44" name="Drills" color="7" fill="1" visible="no" active="yes"/>
-<layer number="45" name="Holes" color="7" fill="1" visible="yes" active="yes"/>
-<layer number="46" name="Milling" color="3" fill="1" visible="yes" active="yes"/>
-<layer number="47" name="Measures" color="7" fill="1" visible="yes" active="yes"/>
+<layer number="45" name="Holes" color="7" fill="1" visible="no" active="yes"/>
+<layer number="46" name="Milling" color="3" fill="1" visible="no" active="yes"/>
+<layer number="47" name="Measures" color="7" fill="1" visible="no" active="yes"/>
 <layer number="48" name="Document" color="7" fill="1" visible="no" active="yes"/>
 <layer number="49" name="Reference" color="7" fill="1" visible="no" active="yes"/>
 <layer number="50" name="dxf" color="7" fill="1" visible="no" active="yes"/>
-<layer number="51" name="tDocu" color="7" fill="1" visible="yes" active="yes"/>
-<layer number="52" name="bDocu" color="7" fill="1" visible="yes" active="yes"/>
+<layer number="51" name="tDocu" color="7" fill="1" visible="no" active="yes"/>
+<layer number="52" name="bDocu" color="7" fill="1" visible="no" active="yes"/>
 <layer number="53" name="tGND_GNDA" color="7" fill="1" visible="no" active="yes"/>
 <layer number="54" name="bGND_GNDA" color="7" fill="1" visible="no" active="yes"/>
@@
 <text x="18.415" y="76.708" size="2.54" layer="25">A</text>
 <text x="79.121" y="76.835" size="2.54" layer="25">B</text>
+<wire x1="11.43" y1="22.86" x2="11.43" y2="15.24" width="0.1524" layer="25"/>
+<wire x1="10.16" y1="21.59" x2="12.7" y2="21.59" width="0.1524" layer="25"/>
+<wire x1="10.16" y1="19.05" x2="12.7" y2="19.05" width="0.1524" layer="25"/>
+<wire x1="10.16" y1="16.51" x2="12.7" y2="16.51" width="0.1524" layer="25"/>
+<text x="11.43" y="13.97" size="1.778" layer="25">1</text>
 </plain>
 <attributes>

Commit message: Autorouted and Manual Layout
Routing:
- net +3V3: vias 1 -> 9
- added copper zone on layer 1, net +3V3
- added copper zone on layer 16, net +3V3
Changed lines of the file:
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@@
 <grid distance="50" unitdist="mil" unit="mil" style="lines" multiple="1" display="yes" altdistance="5" altunitdist="mil" altunit="mil"/>
 <layers>
-<layer number="1" name="Top" color="4" fill="1" visible="no" active="yes"/>
+<layer number="1" name="Top" color="4" fill="1" visible="yes" active="yes"/>
 <layer number="2" name="Route2" color="1" fill="3" visible="no" active="no"/>
 <layer number="3" name="Route3" color="4" fill="3" visible="no" active="no"/>
@@
 <layer number="14" name="Route14" color="1" fill="6" visible="no" active="no"/>
 <layer number="15" name="Route15" color="4" fill="6" visible="no" active="no"/>
-<layer number="16" name="Bottom" color="1" fill="1" visible="no" active="yes"/>
-<layer number="17" name="Pads" color="2" fill="1" visible="no" active="yes"/>
-<layer number="18" name="Vias" color="2" fill="1" visible="no" active="yes"/>
-<layer number="19" name="Unrouted" color="6" fill="1" visible="no" active="yes"/>
-<layer number="20" name="Dimension" color="24" fill="1" visible="no" active="yes"/>
-<layer number="21" name="tPlace" color="7" fill="1" visible="no" active="yes"/>
-<layer number="22" name="bPlace" color="7" fill="1" visible="no" active="yes"/>
-<layer number="23" name="tOrigins" color="15" fill="1" visible="no" active="yes"/>
-<layer number="24" name="bOrigins" color="15" fill="1" visible="no" active="yes"/>
+<layer number="16" name="Bottom" color="1" fill="1" visible="yes" active="yes"/>
+<layer number="17" name="Pads" color="2" fill="1" visible="yes" active="yes"/>
+<layer number="18" name="Vias" color="2" fill="1" visible="yes" active="yes"/>
+<layer number="19" name="Unrouted" color="6" fill="1" visible="yes" active="yes"/>
+<layer number="20" name="Dimension" color="24" fill="1" visible="yes" active="yes"/>
+<layer number="21" name="tPlace" color="7" fill="1" visible="yes" active="yes"/>
+<layer number="22" name="bPlace" color="7" fill="1" visible="yes" active="yes"/>
+<layer number="23" name="tOrigins" color="15" fill="1" visible="yes" active="yes"/>
+<layer number="24" name="bOrigins" color="15" fill="1" visible="yes" active="yes"/>
 <layer number="25" name="tNames" color="7" fill="1" visible="yes" active="yes"/>
-<layer number="26" name="bNames" color="7" fill="1" visible="no" active="yes"/>
-<layer number="27" name="tValues" color="7" fill="1" visible="no" active="yes"/>
-<layer number="28" name="bValues" color="7" fill="1" visible="no" active="yes"/>
+<layer number="26" name="bNames" color="7" fill="1" visible="yes" active="yes"/>
+<layer number="27" name="tValues" color="7" fill="1" visible="yes" active="yes"/>
+<layer number="28" name="bValues" color="7" fill="1" visible="yes" active="yes"/>
 <layer number="29" name="tStop" color="7" fill="3" visible="no" active="yes"/>
 <layer number="30" name="bStop" color="7" fill="6" visible="no" active="yes"/>
@@
 <layer number="37" name="tTest" color="7" fill="1" visible="no" active="yes"/>
 <layer number="38" name="bTest" color="7" fill="1" visible="no" active="yes"/>
-<layer number="39" name="tKeepout" color="4" fill="11" visible="no" active="yes"/>
-<layer number="40" name="bKeepout" color="1" fill="11" visible="no" active="yes"/>
-<layer number="41" name="tRestrict" color="4" fill="10" visible="no" active="yes"/>
-<layer number="42" name="bRestrict" color="1" fill="10" visible="no" active="yes"/>
+<layer number="39" name="tKeepout" color="4" fill="11" visible="yes" active="yes"/>
+<layer number="40" name="bKeepout" color="1" fill="11" visible="yes" active="yes"/>
+<layer number="41" name="tRestrict" color="4" fill="10" visible="yes" active="yes"/>
+<layer number="42" name="bRestrict" color="1" fill="10" visible="yes" active="yes"/>
 <layer number="43" name="vRestrict" color="2" fill="10" visible="no" active="yes"/>
 <layer number="44" name="Drills" color="7" fill="1" visible="no" active="yes"/>
-<layer number="45" name="Holes" color="7" fill="1" visible="no" active="yes"/>
+<layer number="45" name="Holes" color="7" fill="1" visible="yes" active="yes"/>
 <layer number="46" name="Milling" color="3" fill="1" visible="no" active="yes"/>
 <layer number="47" name="Measures" color="7" fill="1" visible="no" active="yes"/>
@@
 <layer number="49" name="Reference" color="7" fill="1" visible="no" active="yes"/>
 <layer number="50" name="dxf" color="7" fill="1" visible="no" active="yes"/>
-<layer number="51" name="tDocu" color="7" fill="1" visible="no" active="yes"/>
-<layer number="52" name="bDocu" color="7" fill="1" visible="no" active="yes"/>
+<layer number="51" name="tDocu" color="7" fill="1" visible="yes" active="yes"/>
+<layer number="52" name="bDocu" color="7" fill="1" visible="yes" active="yes"/>
 <layer number="53" name="tGND_GNDA" color="7" fill="1" visible="no" active="yes"/>
 <layer number="54" name="bGND_GNDA" color="7" fill="1" visible="no" active="yes"/>
@@
 <wire x1="41.275" y1="20.32" x2="41.758" y2="20.32" width="0.1" layer="1"/>
 <wire x1="38.1" y1="24.13" x2="36.83" y2="24" width="0.1" layer="1"/>
+<polygon width="0.3048" layer="1">
+<vertex x="21.59" y="30.48"/>
+<vertex x="21.59" y="21.59"/>
+<vertex x="22.86" y="20.32"/>
+<vertex x="34.29" y="20.32"/>
+<vertex x="34.29" y="30.48"/>
+</polygon>
+<via x="23.495" y="26.035" extent="1-16" drill="0.35"/>
+<via x="23.495" y="27.305" extent="1-16" drill="0.35"/>
+<via x="23.495" y="24.765" extent="1-16" drill="0.35"/>
+<via x="23.495" y="23.495" extent="1-16" drill="0.35"/>
+<via x="22.225" y="23.495" extent="1-16" drill="0.35"/>
+<via x="22.225" y="24.765" extent="1-16" drill="0.35"/>
+<via x="22.225" y="26.035" extent="1-16" drill="0.35"/>
+<via x="22.225" y="27.305" extent="1-16" drill="0.35"/>
+<polygon width="0.3048" layer="16">
+<vertex x="21.59" y="30.48"/>
+<vertex x="21.59" y="21.59"/>
+<vertex x="22.86" y="20.32"/>
+<vertex x="34.29" y="20.32"/>
+<vertex x="34.29" y="30.48"/>
+</polygon>
 </signal>
 <signal name="N$2">
@@
 <via x="48.26" y="48.26" extent="1-16" drill="0.35"/>
 <via x="50.8" y="48.26" extent="1-16" drill="0.35"/>
-<via x="22.225" y="26.035" extent="1-16" drill="0.35"/>
-<via x="22.225" y="24.765" extent="1-16" drill="0.35"/>
-<via x="22.225" y="23.495" extent="1-16" drill="0.35"/>
-<via x="23.495" y="23.495" extent="1-16" drill="0.35"/>
-<via x="23.495" y="24.765" extent="1-16" drill="0.35"/>
-<via x="23.495" y="26.035" extent="1-16" drill="0.35"/>
 <contactref element="R1" pad="1"/>
 <via x="2.54" y="33.02" extent="1-16" drill="0.35"/>
@@
 <via x="24.13" y="13.97" extent="1-16" drill="0.35"/>
 <via x="24.13" y="11.43" extent="1-16" drill="0.35"/>
-<via x="23.495" y="27.305" extent="1-16" drill="0.35"/>
-<via x="22.225" y="27.305" extent="1-16" drill="0.35"/>
 <via x="2.54" y="71.12" extent="1-16" drill="0.35"/>
 <via x="22.86" y="48.26" extent="1-16" drill="0.35"/>
@@
 <contactref element="SV4" pad="20"/>
 <via x="27.94" y="12.827" extent="1-16" drill="1.3208" diameter="2.54"/>
-<via x="34.29" y="21.59" extent="1-16" drill="0.35"/>
-<via x="30.48" y="21.59" extent="1-16" drill="0.35"/>
-<via x="26.67" y="21.59" extent="1-16" drill="0.35"/>
-<via x="22.86" y="21.59" extent="1-16" drill="0.35"/>
 <via x="72.39" y="26.035" extent="1-16" drill="0.35"/>
 <via x="69.215" y="26.035" extent="1-16" drill="0.35"/>
