File: PCB-Eagle/AMP2.brd (EAGLE design)
At the start: 100.4 x 80 mm, 45 parts, among them IC1 LD117AS33TR, IC2 R-78E-0.5, X3 MKDSN1,5/2-5,08

Commit message: Fixed Power Input, added fuses and TCS diodes.
Parts:
- removed L5: 10uH, inductors:DR125
- added L6: fuse, rcl:L5650M
- added TVS: 26Vbi, diode:SMC
- moved D1 17.8 mm to (44.5, 8.89)
Connections:
- removed net ERNIE: D1.A, L5.2
- new net VIN2: D1.C, L6.1
- net +12V: now also L6.2, TVS.C; no longer D1.C
- net GND: now also TVS.A
- net HORST: now also D1.A; no longer L5.1
Routing:
- added copper zone on layer 1, net VIN2
- removed copper zone on layer 1, net ERNIE
Changed lines of the file:
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@@
 <?xml version="1.0" encoding="utf-8"?>
 <!DOCTYPE eagle SYSTEM "eagle.dtd">
-<eagle version="9.6.2">
+<eagle version="9.5.1">
 <drawing>
 <settings>
@@
 <layer number="27" name="tValues" color="7" fill="1" visible="yes" active="yes"/>
 <layer number="28" name="bValues" color="7" fill="1" visible="yes" active="yes"/>
-<layer number="29" name="tStop" color="7" fill="3" visible="no" active="yes"/>
+<layer number="29" name="tStop" color="7" fill="3" visible="yes" active="yes"/>
 <layer number="30" name="bStop" color="7" fill="6" visible="no" active="yes"/>
 <layer number="31" name="tCream" color="7" fill="4" visible="no" active="yes"/>
@@
 <layer number="45" name="Holes" color="7" fill="1" visible="yes" active="yes"/>
 <layer number="46" name="Milling" color="3" fill="1" visible="no" active="yes"/>
-<layer number="47" name="Measures" color="7" fill="1" visible="no" active="yes"/>
+<layer number="47" name="Measures" color="7" fill="1" visible="yes" active="yes"/>
 <layer number="48" name="Document" color="7" fill="1" visible="no" active="yes"/>
 <layer number="49" name="Reference" color="7" fill="1" visible="no" active="yes"/>
@@
 </layers>
 <board>
+<fusionsync huburn="a.cGVyc29uYWw6dWUyOWM4MzJj" projecturn="a.cGVyc29uYWw6dWUyOWM4MzJjIzIwMTkwNzE5MjA0NDAwNTMx" f3durn="urn:adsk.wipprod:dm.lineage:TYoVdYiKR_a4npLLLZPksw" pcbguid="8fff58e3-5e0d-4c8e-90f4-56d0cea54fcf" lastpulledtime="" lastsyncedchangeguid="b05b3e7b-003b-4976-0f22-fc1d69745e30"/>
 <plain>
 <wire x1="5.08" y1="0" x2="95.25" y2="0" width="0" layer="20"/>
@@
 <wire x1="5.08" y1="12.7" x2="13.97" y2="12.7" width="0.1524" layer="25"/>
 <wire x1="13.97" y1="12.7" x2="13.97" y2="25.4" width="0.1524" layer="25"/>
-<text x="96.52" y="11.43" size="1.778" layer="25" rot="R90">GND</text>
-<text x="96.52" y="17.78" size="1.778" layer="25" rot="R90">6-26V</text>
+<text x="27.94" y="3.81" size="1.778" layer="25" rot="R180">GND</text>
+<text x="36.83" y="3.81" size="1.778" layer="25" rot="R180">6-26V</text>
 <text x="33.401" y="15.367" size="1.016" layer="25">GND</text>
 <text x="18.034" y="15.367" size="1.016" layer="25">+12V</text>
@@
 <wire x1="13.081" y1="5.08" x2="13.081" y2="4.953" width="0.1524" layer="25"/>
 <wire x1="13.081" y1="4.953" x2="13.208" y2="4.953" width="0.1524" layer="25"/>
-<wire x1="55.245" y1="21.717" x2="55.245" y2="8.509" width="0.4064" layer="25"/>
-<text x="56.007" y="4.699" size="1.778" layer="25" rot="R90">red</text>
+<wire x1="55.245" y1="21.717" x2="55.245" y2="12.319" width="0.4064" layer="25"/>
+<text x="54.737" y="12.319" size="1.778" layer="25" rot="R90">red</text>
 <text x="62.865" y="14.478" size="1.4224" layer="25" rot="R90">(5V)</text>
 <text x="53.594" y="19.431" size="1.778" layer="25">1</text>
@@
 <wire x1="10.16" y1="16.51" x2="12.7" y2="16.51" width="0.1524" layer="25"/>
 <text x="11.43" y="13.97" size="1.778" layer="25">1</text>
+<polygon width="0.2032" layer="29">
+<vertex x="52.07" y="11.43"/>
+<vertex x="55.88" y="11.43"/>
+<vertex x="55.88" y="6.35"/>
+<vertex x="52.07" y="6.35"/>
+</polygon>
+<polygon width="0.2032" layer="29">
+<vertex x="58.42" y="11.43"/>
+<vertex x="62.23" y="11.43"/>
+<vertex x="62.23" y="6.35"/>
+<vertex x="58.42" y="6.35"/>
+</polygon>
+<dimension x1="53.086" y1="5.08" x2="61.722" y2="5.08" x3="57.404" y3="0" textsize="2.54" layer="47"/>
 </plain>
 <attributes>
@@
 <attribute name="SPICEPREFIX" value="R" x="19.812" y="5.842" size="10.16" layer="27" font="vector" rot="R270" display="off"/>
 </element>
-<element name="L5" library="inductors" library_urn="urn:adsk.eagle:library:243" package="DR125" package3d_urn="urn:adsk.eagle:package:15121/1" value="10uH" x="46.99" y="8.89" smashed="yes">
-<attribute name="NAME" x="44.49" y="11.89" size="1.27" layer="25"/>
-<attribute name="POPULARITY" value="1" x="46.99" y="8.89" size="1.778" layer="27" display="off"/>
-<attribute name="SPICEPREFIX" value="L" x="46.99" y="8.89" size="1.778" layer="27" display="off"/>
-<attribute name="VALUE" x="43.99" y="4.39" size="1.27" layer="27"/>
-</element>
-<element name="D1" library="diode" library_urn="urn:adsk.eagle:library:210" package="SMC" package3d_urn="urn:adsk.eagle:package:43425/2" value="" x="62.23" y="8.89" smashed="yes" rot="R180">
-<attribute name="NAME" x="65.689" y="5.531" size="1.27" layer="25" rot="R180"/>
-<attribute name="POPULARITY" value="1" x="62.23" y="8.89" size="1.778" layer="27" rot="R180" display="off"/>
-<attribute name="VALUE" x="65.689" y="13.519" size="1.27" layer="27" rot="R180"/>
+<element name="D1" library="diode" library_urn="urn:adsk.eagle:library:210" package="SMC" package3d_urn="urn:adsk.eagle:package:43425/2" value="" x="44.45" y="8.89" smashed="yes" rot="R180">
+<attribute name="NAME" x="47.909" y="5.531" size="1.27" layer="25" rot="R180"/>
+<attribute name="POPULARITY" value="1" x="44.45" y="8.89" size="1.778" layer="27" rot="R180" display="off"/>
+<attribute name="VALUE" x="47.909" y="13.519" size="1.27" layer="27" rot="R180"/>
 </element>
 <element name="SJ2" library="jumper" library_urn="urn:adsk.eagle:library:252" package="SJ" package3d_urn="urn:adsk.eagle:package:15471/1" value="" x="52.07" y="17.78" smashed="yes">
@@
 <attribute name="POPULARITY" value="41" x="43.18" y="20.32" size="1.778" layer="27" rot="R180" display="off"/>
 <attribute name="SPICEPREFIX" value="R" x="43.18" y="20.32" size="1.778" layer="27" rot="R180" display="off"/>
+</element>
+<element name="L6" library="rcl" library_urn="urn:adsk.eagle:library:334" package="L5650M" package3d_urn="urn:adsk.eagle:package:23487/2" value="fuse" x="57.15" y="8.89" smashed="yes">
+<attribute name="MOUSER" value="650-ASMDC300F/24-2" x="57.15" y="8.89" size="2.54" layer="27" display="off"/>
+<attribute name="NAME" x="55.245" y="11.43" size="1.27" layer="25"/>
+<attribute name="POPULARITY" value="0" x="57.15" y="8.89" size="2.54" layer="27" display="off"/>
+<attribute name="SPICEPREFIX" value="L" x="57.15" y="8.89" size="2.54" layer="27" display="off"/>
+<attribute name="VALUE" x="55.245" y="3.81" size="1.27" layer="27"/>
+</element>
+<element name="TVS" library="diode" library_urn="urn:adsk.eagle:library:210" package="SMC" package3d_urn="urn:adsk.eagle:package:43425/2" value="26Vbi" x="91.44" y="19.05" smashed="yes">
+<attribute name="NAME" x="90.551" y="22.479" size="1.27" layer="25"/>
+<attribute name="POPULARITY" value="1" x="91.44" y="19.05" size="2.54" layer="27" display="off"/>
+<attribute name="VALUE" x="89.281" y="14.351" size="1.27" layer="27"/>
 </element>
 </elements>
@@
 <via x="20.32" y="44.45" extent="1-16" drill="0.35"/>
 <polygon width="0.4064" layer="1">
-<vertex x="63.5238125" y="12.827"/>
-<vertex x="64.008" y="5.08"/>
+<vertex x="58.928" y="12.9778125"/>
+<vertex x="58.928" y="5.08"/>
 <vertex x="82.55" y="5.08"/>
 <vertex x="89.154" y="11.684"/>
@@
 <via x="71.501" y="6.985" extent="1-16" drill="0.35"/>
 <via x="75.311" y="6.985" extent="1-16" drill="0.35"/>
-<contactref element="D1" pad="C"/>
+<contactref element="L6" pad="2"/>
+<contactref element="TVS" pad="C"/>
 </signal>
 <signal name="+3V3">
@@
 <via x="97.79" y="13.97" extent="1-16" drill="0.35"/>
 <via x="88.9" y="10.16" extent="1-16" drill="0.35"/>
-<via x="95.25" y="17.78" extent="1-16" drill="0.35"/>
 <via x="96.52" y="10.16" extent="1-16" drill="0.35"/>
 <via x="93.98" y="13.97" extent="1-16" drill="0.35"/>
@@
 <via x="22.86" y="36.83" extent="1-16" drill="0.35"/>
 <via x="19.05" y="36.83" extent="1-16" drill="0.35"/>
+<contactref element="TVS" pad="A"/>
 </signal>
 <signal name="SDA">
@@
 <wire x1="19.812" y1="4.42" x2="16.129" y2="4.42" width="1.016" layer="1"/>
 </signal>
-<signal name="ERNIE">
-<polygon width="0.4064" layer="1">
-<vertex x="49.276" y="12.7"/>
-<vertex x="49.276" y="5.08"/>
-<vertex x="60.452" y="5.08"/>
-<vertex x="60.452" y="12.7"/>
-</polygon>
-<contactref element="D1" pad="A"/>
-<contactref element="L5" pad="2"/>
-</signal>
 <signal name="HORST">
 <contactref element="X3" pad="2"/>
@@
 <vertex x="30.48" y="12.7"/>
 <vertex x="30.48" y="5.08"/>
-<vertex x="44.704" y="5.08"/>
-<vertex x="44.704" y="12.7"/>
+<vertex x="43.434" y="5.08"/>
+<vertex x="43.434" y="12.7"/>
 </polygon>
-<contactref element="L5" pad="1"/>
 <via x="33.02" y="12.827" extent="1-16" drill="1.3208" diameter="2.54"/>
 <wire x1="33.02" y1="12.827" x2="33.02" y2="9.0631" width="2.032" layer="16"/>
 <wire x1="33.02" y1="9.0631" x2="32.9989" y2="9.042" width="2.032" layer="16"/>
+<contactref element="D1" pad="A"/>
 </signal>
 <signal name="N$14">
@@
 <contactref element="FAULT" pad="C"/>
 <wire x1="46.838" y1="20.32" x2="44.602" y2="20.32" width="0.1" layer="1"/>
+</signal>
+<signal name="VIN2">
+<contactref element="L6" pad="1"/>
+<contactref element="D1" pad="C"/>
+<polygon width="0.4064" layer="1">
+<vertex x="45.466" y="12.7"/>
+<vertex x="45.466" y="5.08"/>
+<vertex x="55.372" y="5.08"/>
+<vertex x="55.372" y="12.7"/>
+</polygon>
 </signal>
 </signals>
@@
 </note>
 <note version="8.3" severity="warning">
+Since Version 8.3, EAGLE supports Fusion synchronisation.
+This feature will not be available in this version and saving
+the document will break the link to the Fusion PCB feature.
+</note>
+<note version="8.3" severity="warning">
