File: PCB-Eagle/AMP2.brd (EAGLE design)
At the start: 100.4 x 80 mm, 46 parts, among them IC1 LD117AS33TR, IC2 R-78E-0.5, X3 MKDSN1,5/2-5,08

Commit message: Added brown out, 3D models...
Parts:
- removed LED1: (no value), led:1206
- added C20, C22: .1u, rcl:C0603
- added IC3: TL77005ACD, linear:SO08
- added PWR: (no value), led:SML0805
- added R3, R4: 10k, rcl:R0603
- C10, C11, C13, C16, C9: device rcl:C1206 -> rcl:C0603
- FAULT: device led:1206 -> led:SML0805
- R1, R2, R5, R6: device rcl:R1206 -> rcl:R0603
- TVS: value 26Vbi -> 24Vbi
- moved FAULT 30.5 mm to (19.3, 10.8), turned to 0 degrees
- moved TVS 26.7 mm to (67.3, 7.62), turned to 270 degrees
- moved R2 24.7 mm to (19.6, 13.1)
- moved R1 8.12 mm to (16.1, 13.1), turned to 180 degrees
- moved C10 8.00 mm to (48.6, 29.6), turned to 180 degrees
- moved C12 3.50 mm to (34.4, 22.9), turned to 180 degrees
- moved R6 2.92 mm to (43.2, 29.6)
- moved R5 2.54 mm to (43.2, 31.8)
- moved SJ2 1.80 mm to (53.3, 16.5)
- moved C9 1.80 mm to (55.9, 34.3)
- moved C11 1.27 mm to (43.2, 34.3)
Connections:
- net HORST renamed VIN
- new net N$18: IC3.7, R3.1
- new net N$19: IC3.6, R4.2
- new net N$20: C20.2, IC3.1
- new net N$21: C22.2, IC3.3
- new net RESIN: IC3.2, SV4.3
- net +12V: now also R3.2
- net +3V3: now also PWR.C; no longer LED1.C
- net +5V: now also IC3.8
- net GND: now also C20.1, C22.1, IC3.4, R4.1
- net N$13: now also PWR.A; no longer LED1.A
- net PDN: now also IC3.5; no longer SV4.3
Routing:
- net +12V: track 2.88 -> 42.0 mm
- net ADR/FAULT: track 40.1 -> 71.6 mm
- net +3V3: track 65.5 -> 47.6 mm, vias 9 -> 12
- net RESIN: track 0.00 -> 16.5 mm
- net N$15: track 18.4 -> 7.08 mm, vias 2 -> 0
- net N$19: track 0.00 -> 6.42 mm
- net PDN: track 33.1 -> 27.3 mm
- net +5V: track 46.8 -> 52.0 mm
- net N$18: track 0.00 -> 5.01 mm
- net N$21: track 0.00 -> 3.60 mm
- net SDA: track 37.1 -> 33.5 mm
- net SCL: track 38.6 -> 35.2 mm
- net LRCLK: track 39.9 -> 36.7 mm, vias 0 -> 1
- net N$20: track 0.00 -> 2.58 mm
- net N$16: track 5.77 -> 3.92 mm
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Other:
- outline, holes or cut-outs redrawn
- board text added: "9-26V"
- board text removed: "6-26V"
- board text removed: "power2header >"

Commit message: Eagle is a mess. Any capable developers left @ ADSK ?
Parts:
- L6: value fuse -> Fuse
Routing:
- net ADR/FAULT: track 71.6 -> 70.9 mm

Commit message: LED 1206.
Parts:
- removed FAULT, PWR: (no value), led:SML0805
- added FAULT----, PWR-----: (no value), led:1206
- R1, R2: value 220 -> 2.2k
- moved C6 4.79 mm to (46.0, 69.8), turned to 0 degrees
- moved C5 4.69 mm to (22.7, 69.8), turned to 180 degrees
- moved C7 4.58 mm to (77.5, 69.8), turned to 0 degrees
- moved C8 4.58 mm to (54.6, 69.8), turned to 180 degrees
- moved R1 0.38 mm to (15.7, 13.1)
Connections:
- net +3V3: now also PWR-----.C; no longer PWR.C
- net ADR/FAULT: now also FAULT----.A; no longer FAULT.A
- net N$13: now also PWR-----.A; no longer PWR.A
- net N$17: now also FAULT----.C; no longer FAULT.C
Routing:
- net N$10: track 14.1 -> 16.6 mm
- net N$1: track 14.0 -> 16.4 mm
- net N$12: track 14.0 -> 16.2 mm
- net N$11: track 14.1 -> 16.2 mm

Commit message: Cosmetics..
Parts:
- added R7, R8, R9: 47, rcl:R0603
- TVS: value 24Vbi -> 26Vbi
- moved C10 2.11 mm to (47.5, 31.4), turned to 90 degrees
Connections:
- new net N$22: R7.1, U$1.6
- new net N$23: R8.1, U$1.7
- new net N$24: R9.1, U$1.8
- net LRCLK: now also R7.2; no longer U$1.6
- net SCLK: now also R8.2; no longer U$1.7
- net SDIN: now also R9.2; no longer U$1.8
Routing:
- net N$22: track 0.00 -> 13.3 mm
- net N$23: track 0.00 -> 11.0 mm
- net SCLK: track 30.8 -> 21.1 mm
- net LRCLK: track 36.7 -> 27.1 mm
- net SDIN: track 31.5 -> 22.8 mm
- net N$24: track 0.00 -> 8.66 mm
- net N$15: track 7.08 -> 4.16 mm
- net ADR/FAULT: track 70.6 -> 72.7 mm
- net +12V: vias 43 -> 52
Other:
- board text added: "9-25V"
- board text removed: "9-26V"
