File: PCB-Eagle/AMP2.sch (EAGLE design)
At the start: 16 parts, among them IC1 LD117AS33TR

Commit message: Added Terminals 2...
Parts:
- added X1, X2, X3: MKDSN1,5/2-5,08, con-phoenix-508:MKDSN1,5/2-5,08
Connections:
- net +12V: now also IC1.IN, X3-2.KL
- net +3V3: now also IC1.OUT
- net GND: now also IC1.ADJ, X3-1.KL
- net N$1: now also X1-1.KL
- net N$10: now also X1-2.KL
- net N$11: now also X2-2.KL
- net N$12: now also X2-1.KL
Other:
- moved on the sheet: IC1
Changed lines of the file:
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@@
 <part name="GND2" library="supply1" library_urn="urn:adsk.eagle:library:371" deviceset="GND" device=""/>
 <part name="GND3" library="supply1" library_urn="urn:adsk.eagle:library:371" deviceset="GND" device=""/>
+<part name="X1" library="con-phoenix-508" library_urn="urn:adsk.eagle:library:176" deviceset="MKDSN1,5/2-5,08" device="" package3d_urn="urn:adsk.eagle:package:9630/1"/>
+<part name="X2" library="con-phoenix-508" library_urn="urn:adsk.eagle:library:176" deviceset="MKDSN1,5/2-5,08" device="" package3d_urn="urn:adsk.eagle:package:9630/1"/>
+<part name="X3" library="con-phoenix-508" library_urn="urn:adsk.eagle:library:176" deviceset="MKDSN1,5/2-5,08" device="" package3d_urn="urn:adsk.eagle:package:9630/1"/>
+<part name="P+2" library="supply1" library_urn="urn:adsk.eagle:library:371" deviceset="+12V" device=""/>
+<part name="GND4" library="supply1" library_urn="urn:adsk.eagle:library:371" deviceset="GND" device=""/>
+<part name="GND5" library="supply1" library_urn="urn:adsk.eagle:library:371" deviceset="GND" device=""/>
+<part name="+3V2" library="supply1" library_urn="urn:adsk.eagle:library:371" deviceset="+3V3" device=""/>
 </parts>
 <sheets>
@@
 <attribute name="VALUE" x="7.62" y="68.58" size="1.778" layer="96" rot="R90"/>
 </instance>
-<instance part="IC1" gate="G$1" x="22.86" y="93.98" smashed="yes">
-<attribute name="NAME" x="25.4" y="86.36" size="1.778" layer="95"/>
-<attribute name="VALUE" x="25.4" y="83.82" size="1.778" layer="96"/>
+<instance part="IC1" gate="G$1" x="43.18" y="106.68" smashed="yes">
+<attribute name="NAME" x="45.72" y="99.06" size="1.778" layer="95"/>
+<attribute name="VALUE" x="45.72" y="96.52" size="1.778" layer="96"/>
 </instance>
 <instance part="C1" gate="G$1" x="124.46" y="55.88" smashed="yes" rot="R90">
@@
 <attribute name="VALUE" x="175.26" y="55.88" size="1.778" layer="96"/>
 </instance>
-<instance part="GND2" gate="1" x="210.82" y="58.42" smashed="yes">
-<attribute name="VALUE" x="208.28" y="55.88" size="1.778" layer="96"/>
+<instance part="GND2" gate="1" x="177.8" y="10.16" smashed="yes">
+<attribute name="VALUE" x="175.26" y="7.62" size="1.778" layer="96"/>
 </instance>
 <instance part="GND3" gate="1" x="124.46" y="15.24" smashed="yes">
 <attribute name="VALUE" x="121.92" y="12.7" size="1.778" layer="96"/>
+</instance>
+<instance part="X1" gate="-1" x="193.04" y="99.06" smashed="yes">
+<attribute name="NAME" x="196.088" y="98.171" size="1.778" layer="95"/>
+<attribute name="VALUE" x="190.5" y="95.377" size="1.778" layer="96"/>
+</instance>
+<instance part="X1" gate="-2" x="193.04" y="88.9" smashed="yes">
+<attribute name="NAME" x="196.088" y="88.011" size="1.778" layer="95"/>
+<attribute name="VALUE" x="190.5" y="85.217" size="1.778" layer="96"/>
+</instance>
+<instance part="X2" gate="-1" x="193.04" y="68.58" smashed="yes">
+<attribute name="NAME" x="196.088" y="67.691" size="1.778" layer="95"/>
+<attribute name="VALUE" x="190.5" y="64.897" size="1.778" layer="96"/>
+</instance>
+<instance part="X2" gate="-2" x="193.04" y="78.74" smashed="yes">
+<attribute name="NAME" x="196.088" y="77.851" size="1.778" layer="95"/>
+<attribute name="VALUE" x="190.5" y="75.057" size="1.778" layer="96"/>
+</instance>
+<instance part="X3" gate="-1" x="17.78" y="101.6" smashed="yes" rot="R180">
+<attribute name="NAME" x="14.732" y="102.489" size="1.778" layer="95" rot="R180"/>
+<attribute name="VALUE" x="20.32" y="105.283" size="1.778" layer="96" rot="R180"/>
+</instance>
+<instance part="X3" gate="-2" x="17.78" y="106.68" smashed="yes" rot="R180">
+<attribute name="NAME" x="14.732" y="107.569" size="1.778" layer="95" rot="R180"/>
+<attribute name="VALUE" x="20.32" y="110.363" size="1.778" layer="96" rot="R180"/>
+</instance>
+<instance part="P+2" gate="1" x="25.4" y="111.76" smashed="yes">
+<attribute name="VALUE" x="22.86" y="106.68" size="1.778" layer="96" rot="R90"/>
+</instance>
+<instance part="GND4" gate="1" x="43.18" y="88.9" smashed="yes">
+<attribute name="VALUE" x="40.64" y="86.36" size="1.778" layer="96"/>
+</instance>
+<instance part="GND5" gate="1" x="25.4" y="88.9" smashed="yes">
+<attribute name="VALUE" x="22.86" y="86.36" size="1.778" layer="96"/>
+</instance>
+<instance part="+3V2" gate="G$1" x="60.96" y="111.76" smashed="yes">
+<attribute name="VALUE" x="58.42" y="106.68" size="1.778" layer="96" rot="R90"/>
 </instance>
 </instances>
@@
 <junction x="45.72" y="66.04"/>
 </segment>
+<segment>
+<pinref part="X3" gate="-2" pin="KL"/>
+<wire x1="20.32" y1="106.68" x2="25.4" y2="106.68" width="0.1524" layer="91"/>
+<pinref part="P+2" gate="1" pin="+12V"/>
+<wire x1="25.4" y1="106.68" x2="25.4" y2="109.22" width="0.1524" layer="91"/>
+<pinref part="IC1" gate="G$1" pin="IN"/>
+<wire x1="35.56" y1="106.68" x2="25.4" y2="106.68" width="0.1524" layer="91"/>
+<junction x="25.4" y="106.68"/>
+</segment>
 </net>
 <net name="+3V3" class="0">
@@
 <junction x="22.86" y="55.88"/>
 </segment>
+<segment>
+<pinref part="IC1" gate="G$1" pin="OUT"/>
+<pinref part="+3V2" gate="G$1" pin="+3V3"/>
+<wire x1="50.8" y1="106.68" x2="60.96" y2="106.68" width="0.1524" layer="91"/>
+<wire x1="60.96" y1="106.68" x2="60.96" y2="109.22" width="0.1524" layer="91"/>
+</segment>
 </net>
 <net name="N$2" class="0">
@@
 <pinref part="L1" gate="G$1" pin="2"/>
 <wire x1="162.56" y1="99.06" x2="160.02" y2="99.06" width="0.1524" layer="91"/>
-<wire x1="182.88" y1="99.06" x2="162.56" y2="99.06" width="0.1524" layer="91"/>
+<wire x1="190.5" y1="99.06" x2="162.56" y2="99.06" width="0.1524" layer="91"/>
 <junction x="162.56" y="99.06"/>
+<pinref part="X1" gate="-1" pin="KL"/>
 </segment>
 </net>
@@
 <pinref part="L2" gate="G$1" pin="2"/>
 <wire x1="165.1" y1="88.9" x2="162.56" y2="88.9" width="0.1524" layer="91"/>
-<wire x1="185.42" y1="88.9" x2="165.1" y2="88.9" width="0.1524" layer="91"/>
+<wire x1="190.5" y1="88.9" x2="165.1" y2="88.9" width="0.1524" layer="91"/>
 <junction x="165.1" y="88.9"/>
+<pinref part="X1" gate="-2" pin="KL"/>
 </segment>
 </net>
@@
 <pinref part="L3" gate="G$1" pin="2"/>
 <wire x1="167.64" y1="78.74" x2="165.1" y2="78.74" width="0.1524" layer="91"/>
-<wire x1="187.96" y1="78.74" x2="167.64" y2="78.74" width="0.1524" layer="91"/>
+<pinref part="X2" gate="-2" pin="KL"/>
+<wire x1="167.64" y1="78.74" x2="190.5" y2="78.74" width="0.1524" layer="91"/>
 <junction x="167.64" y="78.74"/>
 </segment>
@@
 <pinref part="L4" gate="G$1" pin="2"/>
 <wire x1="170.18" y1="68.58" x2="167.64" y2="68.58" width="0.1524" layer="91"/>
-<wire x1="190.5" y1="68.58" x2="170.18" y2="68.58" width="0.1524" layer="91"/>
+<pinref part="X2" gate="-1" pin="KL"/>
+<wire x1="170.18" y1="68.58" x2="190.5" y2="68.58" width="0.1524" layer="91"/>
 <junction x="170.18" y="68.58"/>
 </segment>
@@
 </segment>
 </net>
-<net name="N$15" class="0">
-<segment>
-<wire x1="190.5" y1="91.44" x2="182.88" y2="91.44" width="0.1524" layer="91"/>
-</segment>
-</net>
-<net name="N$16" class="0">
-<segment>
-<wire x1="193.04" y1="81.28" x2="185.42" y2="81.28" width="0.1524" layer="91"/>
-</segment>
-</net>
-<net name="N$17" class="0">
-<segment>
-<wire x1="195.58" y1="71.12" x2="187.96" y2="71.12" width="0.1524" layer="91"/>
-</segment>
-</net>
-<net name="N$18" class="0">
-<segment>
-<wire x1="198.12" y1="60.96" x2="190.5" y2="60.96" width="0.1524" layer="91"/>
-</segment>
-</net>
 <net name="GND" class="0">
-<segment>
-<pinref part="GND2" gate="1" pin="GND"/>
-<wire x1="210.82" y1="60.96" x2="208.28" y2="60.96" width="0.1524" layer="91"/>
-<wire x1="210.82" y1="60.96" x2="210.82" y2="71.12" width="0.1524" layer="91"/>
-<junction x="210.82" y="60.96"/>
-<wire x1="210.82" y1="71.12" x2="205.74" y2="71.12" width="0.1524" layer="91"/>
-<wire x1="210.82" y1="71.12" x2="210.82" y2="81.28" width="0.1524" layer="91"/>
-<junction x="210.82" y="71.12"/>
-<wire x1="210.82" y1="81.28" x2="203.2" y2="81.28" width="0.1524" layer="91"/>
-<wire x1="210.82" y1="81.28" x2="210.82" y2="91.44" width="0.1524" layer="91"/>
-<junction x="210.82" y="81.28"/>
-<wire x1="210.82" y1="91.44" x2="200.66" y2="91.44" width="0.1524" layer="91"/>
-</segment>
 <segment>
 <pinref part="GND1" gate="1" pin="GND"/>
@@
 <wire x1="124.46" y1="40.64" x2="116.84" y2="40.64" width="0.1524" layer="91"/>
 </segment>
-</net>
+<segment>
+<pinref part="X3" gate="-1" pin="KL"/>
+<wire x1="20.32" y1="101.6" x2="25.4" y2="101.6" width="0.1524" layer="91"/>
+<pinref part="GND5" gate="1" pin="GND"/>
+<wire x1="25.4" y1="101.6" x2="25.4" y2="91.44" width="0.1524" layer="91"/>
+</segment>
+<segment>
+<pinref part="GND4" gate="1" pin="GND"/>
+<pinref part="IC1" gate="G$1" pin="ADJ"/>
+<wire x1="43.18" y1="91.44" x2="43.18" y2="99.06" width="0.1524" layer="91"/>
+</segment>
+</net>

Commit message: longer todo list :(
Parts:
- added SV1: (no value), con-lsta:FE05-1
- added SV2: (no value), con-lsta:FE08-2
Connections:
- new net SCL: SV1.4, U$1.SCL
- new net SDA: SV1.3, U$1.SDA
- net GND: now also SV1.5
Changed lines of the file:
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@@
 <part name="GND5" library="supply1" library_urn="urn:adsk.eagle:library:371" deviceset="GND" device=""/>
 <part name="+3V2" library="supply1" library_urn="urn:adsk.eagle:library:371" deviceset="+3V3" device=""/>
+<part name="SV1" library="con-lsta" library_urn="urn:adsk.eagle:library:161" deviceset="FE05-1" device="" package3d_urn="urn:adsk.eagle:package:8190/1"/>
+<part name="SV2" library="con-lsta" library_urn="urn:adsk.eagle:library:161" deviceset="FE08-2" device="" package3d_urn="urn:adsk.eagle:package:8174/1"/>
 </parts>
 <sheets>
@@
 <instance part="+3V2" gate="G$1" x="60.96" y="111.76" smashed="yes">
 <attribute name="VALUE" x="58.42" y="106.68" size="1.778" layer="96" rot="R90"/>
+</instance>
+<instance part="SV1" gate="G$1" x="193.04" y="27.94" smashed="yes" rot="R180">
+<attribute name="VALUE" x="194.31" y="38.1" size="1.778" layer="96" rot="R180"/>
+<attribute name="NAME" x="194.31" y="19.558" size="1.778" layer="95" rot="R180"/>
+</instance>
+<instance part="SV2" gate="G$1" x="149.86" y="22.86" smashed="yes">
+<attribute name="VALUE" x="146.05" y="10.16" size="1.778" layer="96"/>
+<attribute name="NAME" x="146.05" y="36.322" size="1.778" layer="95"/>
 </instance>
 </instances>
@@
 <wire x1="43.18" y1="91.44" x2="43.18" y2="99.06" width="0.1524" layer="91"/>
 </segment>
-</net>
+<segment>
+<pinref part="GND2" gate="1" pin="GND"/>
+<wire x1="177.8" y1="12.7" x2="177.8" y2="22.86" width="0.1524" layer="91"/>
+<pinref part="SV1" gate="G$1" pin="5"/>
+<wire x1="177.8" y1="22.86" x2="185.42" y2="22.86" width="0.1524" layer="91"/>
+</segment>
+</net>
+<net name="SDA" class="0">
+<segment>
+<pinref part="U$1" gate="G$1" pin="SDA"/>
+<wire x1="48.26" y1="43.18" x2="33.02" y2="43.18" width="0.1524" layer="91"/>
+<label x="35.56" y="43.18" size="1.778" layer="95"/>
+</segment>
+<segment>
+<pinref part="SV1" gate="G$1" pin="3"/>
+<wire x1="185.42" y1="27.94" x2="170.18" y2="27.94" width="0.1524" layer="91"/>
+<label x="172.72" y="27.94" size="1.778" layer="95"/>
+</segment>
+</net>
+<net name="SCL" class="0">
+<segment>
+<pinref part="U$1" gate="G$1" pin="SCL"/>
+<wire x1="48.26" y1="40.64" x2="33.02" y2="40.64" width="0.1524" layer="91"/>
+<label x="35.56" y="40.64" size="1.778" layer="95"/>
+</segment>
+<segment>
+<pinref part="SV1" gate="G$1" pin="4"/>
+<wire x1="185.42" y1="25.4" x2="170.18" y2="25.4" width="0.1524" layer="91"/>
+<label x="172.72" y="25.4" size="1.778" layer="95"/>
+</segment>
+</net>

Commit message: Removed Pi header, added power filter.
Parts:
- added C10, C9: 1u, rcl:C-EUC1206
- added C11, C13, C16: .1u, rcl:C-EUC1206
- added C12: 10u, rcl:C-EUC1210
- added C14, C15, C17, C18, C19, C21: 220u, rcl:CPOL-EU150CLZ-1010
- added D1: (no value), diode:SCHOTTKY-DIODESMC
- added H1, H2, H3, H4: MOUNT-HOLE3.2, holes:MOUNT-HOLE3.2
- added IC2: R-78E-0.5, linear:788TV
- added L5: 10uH, inductors:DR125
- added LED1: (no value), led:LEDSMT1206
- added R1: 220, rcl:R-EU_R1206
- added SJ1, SJ2: (no value), jumper:SJ
- added SV3: (no value), con-lsta:FE08-1
- C5, C6, C7, C8: value 2.2n -> 680n
- R5: value (none) -> 4.7k
- R6: value (none) -> 10k
- renumbered X1 to OUT-L, X2 to OUT-R
Connections:
- new net +5V: IC1.IN, IC2.VO, SJ2.1, SV3.3, SV3.4
- new net ADR/FAULT: R5.1, SV1.1, U$1.ADR/FAULT
- new net ERNIE: D1.A, L5.2
- new net HORST: L5.1, X3-2.KL
- new net LRCLK: SV2.9, U$1.LRCLK
- new net N$15: C10.2, U$1.VR_DIG
- new net N$16: C9.2, U$1.AVDD
- new net N$19: SJ2.2, SV2.1
- new net PDN: R6.1, SJ1.1, SV1.2, U$1.PDN
- new net SCLK: SV2.7, U$1.SCLK
- new net SDIN: SV2.3, U$1.SDIN
- new net SDOUT: SV2.5, U$1.SDOUT
- net +12V: now also C13.2, C14.+, C15.+, C16.2, C17.+, C18.+, C19.+, C21.+, D1.C, IC2.VI, SV3.1, SV3.2; no longer IC1.IN, X3-2.KL
- net +3V3: now also C11.2, C12.2, LED1.C, SV3.5, SV3.6
- net GND: now also C10.1, C11.1, C12.1, C13.1, C14.-, C15.-, C16.1, C17.-, C18.-, C19.-, C21.-, C9.1, IC2.GND, R1.1, SV2.10, SV2.12, SV2.14, SV2.16, SV2.2, SV2.4, SV2.6, SV2.8, SV3.7, SV3.8; no longer U$1.SDOUT
- net N$13: now also LED1.A, R1.2; no longer R6.1, U$1.PDN
- net N$14: now also SJ1.2, SV2.15; no longer R5.1, U$1.ADR/FAULT
- net SCL: now also SV2.13
- net SDA: now also SV2.11
Other:
- note added: "(MCLK)"
- note added: "R5 for DevAdr 4.7k 15k 47k 120k"
- note added: "oder wi adc/spdif boards"
- note added: "wie adau prog port"
- note added: "wie freedsp ?"
- moved on the sheet: IC1, R5, SV2

Commit message: rev2..
Parts:
- removed SJ1: (no value), jumper:SJ
- removed SV1: (no value), con-lsta:FE05-1
- removed SV2: (no value), con-lsta:FE08-2
- added SV4: (no value), con-lsta:FE10-2
Connections:
- removed net N$19: SJ2.2, SV2.1
- net ADR/FAULT: now also SV4.1; no longer SV1.1
- net GND: now also SV4.10, SV4.12, SV4.14, SV4.16, SV4.18, SV4.20, SV4.6, SV4.8; no longer SV1.5, SV2.10, SV2.12, SV2.14, SV2.16, SV2.2, SV2.4, SV2.6, SV2.8
- net LRCLK: now also SV4.13; no longer SV2.9
- net N$14: now also SJ2.2, SV4.5; no longer SJ1.2, SV2.15
- net PDN: now also SV4.3; no longer SJ1.1, SV1.2
- net SCL: now also SV4.17; no longer SV1.4, SV2.13
- net SCLK: now also SV4.11; no longer SV2.7
- net SDA: now also SV4.15; no longer SV1.3, SV2.11
- net SDIN: now also SV4.7; no longer SV2.3
- net SDOUT: now also SV4.9; no longer SV2.5
Other:
- moved on the sheet: SJ2

Commit message: v02
Parts:
- added FAULT: (no value), led:LEDSMT1206
- added R2: 220, rcl:R-EU_R1206
Connections:
- new net N$17: FAULT.C, R2.1
- net +3V3: now also R2.2
- net ADR/FAULT: now also FAULT.A
Other:
- note added: "(acording datasheet 9.4.2.1 page 34)"
- note added: "The amplified left signal is presented on differential output pair shown as OUT_A+ and OUT_A-,"
- note added: "the amplified right signal is presented on differential output pair shown as OUT_B+ and OUT_B-."
Changed lines of the file:
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@@
 <?xml version="1.0" encoding="utf-8"?>
 <!DOCTYPE eagle SYSTEM "eagle.dtd">
-<eagle version="9.6.1">
+<eagle version="9.6.2">
 <drawing>
 <settings>
@@
 <part name="SJ2" library="jumper" library_urn="urn:adsk.eagle:library:252" deviceset="SJ" device="" package3d_urn="urn:adsk.eagle:package:15471/1"/>
 <part name="SV4" library="con-lsta" library_urn="urn:adsk.eagle:library:161" deviceset="FE10-2" device="" package3d_urn="urn:adsk.eagle:package:8177/1"/>
+<part name="FAULT" library="led" library_urn="urn:adsk.eagle:library:259" deviceset="LED" device="SMT1206" package3d_urn="urn:adsk.eagle:package:15796/2"/>
+<part name="R2" library="rcl" library_urn="urn:adsk.eagle:library:334" deviceset="R-EU_" device="R1206" package3d_urn="urn:adsk.eagle:package:23540/2" value="220"/>
 </parts>
 <sheets>
@@
 <text x="157.48" y="-5.588" size="1.778" layer="97">(MCLK)</text>
 <text x="10.16" y="30.48" size="1.778" layer="97">R5 for DevAdr 4.7k 15k 47k 120k</text>
+<text x="78.74" y="124.46" size="1.778" layer="97">The amplified left signal is presented on differential output pair shown as OUT_A+ and OUT_A-,</text>
+<text x="78.74" y="121.92" size="1.778" layer="97">the amplified right signal is presented on differential output pair shown as OUT_B+ and OUT_B-. </text>
+<text x="78.74" y="119.38" size="1.778" layer="97">(acording datasheet 9.4.2.1 page 34)</text>
 </plain>
 <instances>
@@
 <attribute name="VALUE" x="173.99" y="22.86" size="1.778" layer="96" rot="MR180"/>
 <attribute name="NAME" x="173.99" y="-8.382" size="1.778" layer="95" rot="MR180"/>
+</instance>
+<instance part="FAULT" gate="G$1" x="2.54" y="38.1" smashed="yes" rot="R180">
+<attribute name="NAME" x="-1.016" y="42.672" size="1.778" layer="95" rot="R270"/>
+<attribute name="VALUE" x="-3.175" y="42.672" size="1.778" layer="96" rot="R270"/>
+</instance>
+<instance part="R2" gate="G$1" x="2.54" y="50.8" smashed="yes" rot="R90">
+<attribute name="NAME" x="1.0414" y="46.99" size="1.778" layer="95" rot="R90"/>
+<attribute name="VALUE" x="5.842" y="46.99" size="1.778" layer="96" rot="R90"/>
 </instance>
 </instances>
@@
 <wire x1="20.32" y1="48.26" x2="20.32" y2="55.88" width="0.1524" layer="91"/>
 <junction x="20.32" y="55.88"/>
+<pinref part="R2" gate="G$1" pin="2"/>
+<wire x1="7.62" y1="55.88" x2="2.54" y2="55.88" width="0.1524" layer="91"/>
+<junction x="7.62" y="55.88"/>
 </segment>
 <segment>
@@
 <wire x1="48.26" y1="35.56" x2="20.32" y2="35.56" width="0.1524" layer="91"/>
 <pinref part="R5" gate="G$1" pin="1"/>
-<wire x1="20.32" y1="35.56" x2="10.16" y2="35.56" width="0.1524" layer="91"/>
+<wire x1="20.32" y1="35.56" x2="2.54" y2="35.56" width="0.1524" layer="91"/>
 <wire x1="20.32" y1="35.56" x2="20.32" y2="38.1" width="0.1524" layer="91"/>
 <junction x="20.32" y="35.56"/>
 <label x="33.02" y="35.56" size="1.778" layer="95"/>
+<pinref part="FAULT" gate="G$1" pin="A"/>
 </segment>
 <segment>
@@
 </segment>
 </net>
+<net name="N$17" class="0">
+<segment>
+<pinref part="R2" gate="G$1" pin="1"/>
+<pinref part="FAULT" gate="G$1" pin="C"/>
+<wire x1="2.54" y1="45.72" x2="2.54" y2="43.18" width="0.1524" layer="91"/>
+</segment>
+</net>

Commit message: Fixed Power Input, added fuses and TCS diodes.
Parts:
- removed L5: 10uH, inductors:DR125
- added L6: fuse, rcl:L-EUL5650M
- added TVS: 26Vbi, diode:SCHOTTKY-DIODESMC
Connections:
- removed net ERNIE: D1.A, L5.2
- new net VIN2: D1.C, L6.1
- net +12V: now also L6.2, TVS.C; no longer D1.C
- net GND: now also TVS.A
- net HORST: now also D1.A; no longer L5.1
Other:
- moved on the sheet: D1
