File: PCB-Eagle/AMP2.sch (EAGLE design)
At the start: 51 parts, among them IC1 LD117AS33TR, IC2 R-78E-0.5, IC3 TL77005ACD, X3 MKDSN1,5/2-5,08

Commit message: Eagle is a mess. Any capable developers left @ ADSK ?
Parts:
- L6: value fuse -> Fuse
Changed lines of the file:
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@@
 <part name="FAULT" library="led" library_urn="urn:adsk.eagle:library:259" deviceset="LED" device="SML0805" package3d_urn="urn:adsk.eagle:package:15830/1" override_package3d_urn="urn:adsk.eagle:package:30069147/2" override_package_urn="urn:adsk.eagle:footprint:15683/1"/>
 <part name="R2" library="rcl" library_urn="urn:adsk.eagle:library:334" deviceset="R-EU_" device="R0603" package3d_urn="urn:adsk.eagle:package:23555/3" value="220"/>
-<part name="L6" library="rcl" library_urn="urn:adsk.eagle:library:334" deviceset="L-EU" device="L5650M" package3d_urn="urn:adsk.eagle:package:23487/2" value="fuse">
+<part name="L6" library="rcl" library_urn="urn:adsk.eagle:library:334" deviceset="L-EU" device="L5650M" package3d_urn="urn:adsk.eagle:package:23487/2" value="Fuse">
 <attribute name="MOUSER" value="650-ASMDC300F/24-2"/>
 </part>

Commit message: LED 1206.
Parts:
- removed FAULT, PWR: (no value), led:LEDSML0805
- added FAULT----, PWR-----: (no value), led:LEDSMT1206
- R1, R2: value 220 -> 2.2k
Connections:
- net +3V3: now also PWR-----.C; no longer PWR.C
- net ADR/FAULT: now also FAULT----.A; no longer FAULT.A
- net N$13: now also PWR-----.A; no longer PWR.A
- net N$17: now also FAULT----.C; no longer FAULT.C

Commit message: BOM...
Parts:
- C1, C2, C3, C4: MOUSER (none) -> 80-C1206C224K5R7210
- C10, C9: MOUSER (none) -> 81-GRT188R61H105KE3D
- C11, C13, C16, C20, C22: MOUSER (none) -> 80-C1206C104K5R7210
- C12: MOUSER (none) -> 187-CL32A106KLULNNE
- C14, C15, C17, C18, C19, C21: MOUSER (none) -> 667-EEE-FC1V331AP 667-35SVPK330M
- C5, C6, C7, C8: MOUSER (none) -> 810-C3216X7R1H684K
- D1: MOUSER (none) -> 621-B540C-F
- FAULT----, PWR-----: MOUSER (none) -> 645-599-0220-007F
- IC1: MOUSER (none) -> 621-AZ1117CH2-33TRG1
- IC2: MOUSER (none) -> 919-R-78E5.0-0.5
- IC3: MOUSER (none) -> 595-TL7705AIDR
- L1, L2, L3, L4: MOUSER (none) -> 652-SRU1048-220Y 652-SRU1063A-220Y 652-SRR1260-220M
- R1, R2: MOUSER (none) -> 667-ERJ-3GEYJ222V
- R3, R4, R6: MOUSER (none) -> 667-ERJ-3EKF1002V
- R5: MOUSER (none) -> 667-ERJ-U03J472V
- U$1: MOUSER (none) -> 595-TAS5805MPWP

Commit message: Cosmetics..
Parts:
- added R7, R8, R9: 47, rcl:R-EU_R0603
- TVS: value 24Vbi -> 26Vbi
Connections:
- new net N$22: R7.1, U$1.LRCLK
- new net N$23: R8.1, U$1.SCLK
- new net N$24: R9.1, U$1.SDIN
- net LRCLK: now also R7.2; no longer U$1.LRCLK
- net SCLK: now also R8.2; no longer U$1.SCLK
- net SDIN: now also R9.2; no longer U$1.SDIN
Changed lines of the file:
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@@
 <attribute name="MOUSER" value="650-ASMDC300F/24-2"/>
 </part>
-<part name="TVS" library="diode" library_urn="urn:adsk.eagle:library:210" deviceset="SCHOTTKY-DIODE" device="SMC" package3d_urn="urn:adsk.eagle:package:43425/2" value="24Vbi">
+<part name="TVS" library="diode" library_urn="urn:adsk.eagle:library:210" deviceset="SCHOTTKY-DIODE" device="SMC" package3d_urn="urn:adsk.eagle:package:43425/2" value="26Vbi">
 <attribute name="MOUSER" value="710-824551241"/>
 </part>
@@
 </part>
 <part name="GND18" library="supply1" library_urn="urn:adsk.eagle:library:371" deviceset="GND" device=""/>
+<part name="R7" library="rcl" library_urn="urn:adsk.eagle:library:334" deviceset="R-EU_" device="R0603" package3d_urn="urn:adsk.eagle:package:23555/3" value="47">
+<spice>
+<pinmapping spiceprefix="R">
+<pinmap gate="G$1" pin="1" pinorder="1"/>
+<pinmap gate="G$1" pin="2" pinorder="2"/>
+</pinmapping>
+</spice>
+<attribute name="MOUSER" value="667-ERJ-3EKF1002V "/>
+</part>
+<part name="R8" library="rcl" library_urn="urn:adsk.eagle:library:334" deviceset="R-EU_" device="R0603" package3d_urn="urn:adsk.eagle:package:23555/3" value="47">
+<spice>
+<pinmapping spiceprefix="R">
+<pinmap gate="G$1" pin="1" pinorder="1"/>
+<pinmap gate="G$1" pin="2" pinorder="2"/>
+</pinmapping>
+</spice>
+<attribute name="MOUSER" value="667-ERJ-3EKF1002V "/>
+</part>
+<part name="R9" library="rcl" library_urn="urn:adsk.eagle:library:334" deviceset="R-EU_" device="R0603" package3d_urn="urn:adsk.eagle:package:23555/3" value="47">
+<spice>
+<pinmapping spiceprefix="R">
+<pinmap gate="G$1" pin="1" pinorder="1"/>
+<pinmap gate="G$1" pin="2" pinorder="2"/>
+</pinmapping>
+</spice>
+<attribute name="MOUSER" value="667-ERJ-3EKF1002V "/>
+</part>
 </parts>
 <sheets>
@@
 <text x="137.16" y="38.1" size="1.778" layer="97">oder wi adc/spdif boards</text>
 <text x="157.48" y="-5.588" size="1.778" layer="97">(MCLK)</text>
-<text x="-2.54" y="27.94" size="1.778" layer="97">R5 for DevAdr 4.7k 15k 47k 120k</text>
+<text x="33.02" y="0" size="1.778" layer="97">R5 for DevAdr 4.7k 15k 47k 120k</text>
 <text x="109.22" y="111.76" size="1.778" layer="97">The amplified left signal is presented on differential output pair shown as OUT_A+ and OUT_A-,</text>
 <text x="109.22" y="109.22" size="1.778" layer="97">the amplified right signal is presented on differential output pair shown as OUT_B+ and OUT_B-. </text>
@@
 <instance part="GND18" gate="1" x="33.02" y="83.82" smashed="yes">
 <attribute name="VALUE" x="30.48" y="81.28" size="1.778" layer="96"/>
+</instance>
+<instance part="R7" gate="G$1" x="40.64" y="27.94" smashed="yes" rot="R180">
+<attribute name="NAME" x="44.45" y="26.4414" size="1.778" layer="95" rot="R180"/>
+<attribute name="VALUE" x="44.45" y="31.242" size="1.778" layer="96" rot="R180"/>
+<attribute name="MOUSER" x="40.64" y="27.94" size="1.778" layer="96" rot="R180" display="off"/>
+</instance>
+<instance part="R8" gate="G$1" x="40.64" y="25.4" smashed="yes" rot="R180">
+<attribute name="NAME" x="44.45" y="23.9014" size="1.778" layer="95" rot="R180"/>
+<attribute name="VALUE" x="44.45" y="28.702" size="1.778" layer="96" rot="R180"/>
+<attribute name="MOUSER" x="40.64" y="25.4" size="1.778" layer="96" rot="R180" display="off"/>
+</instance>
+<instance part="R9" gate="G$1" x="40.64" y="22.86" smashed="yes" rot="R180">
+<attribute name="NAME" x="44.45" y="21.3614" size="1.778" layer="95" rot="R180"/>
+<attribute name="VALUE" x="44.45" y="26.162" size="1.778" layer="96" rot="R180"/>
+<attribute name="MOUSER" x="40.64" y="22.86" size="1.778" layer="96" rot="R180" display="off"/>
 </instance>
 </instances>
@@
 <net name="LRCLK" class="0">
 <segment>
-<pinref part="U$1" gate="G$1" pin="LRCLK"/>
-<wire x1="48.26" y1="27.94" x2="35.56" y2="27.94" width="0.1524" layer="91"/>
-<label x="35.56" y="27.94" size="1.778" layer="95"/>
+<wire x1="35.56" y1="27.94" x2="22.86" y2="27.94" width="0.1524" layer="91"/>
+<label x="22.86" y="27.94" size="1.778" layer="95"/>
+<pinref part="R7" gate="G$1" pin="2"/>
 </segment>
 <segment>
@@
 <net name="SCLK" class="0">
 <segment>
-<pinref part="U$1" gate="G$1" pin="SCLK"/>
-<wire x1="48.26" y1="25.4" x2="35.56" y2="25.4" width="0.1524" layer="91"/>
-<label x="35.56" y="25.4" size="1.778" layer="95"/>
+<wire x1="35.56" y1="25.4" x2="22.86" y2="25.4" width="0.1524" layer="91"/>
+<label x="22.86" y="25.4" size="1.778" layer="95"/>
+<pinref part="R8" gate="G$1" pin="2"/>
 </segment>
 <segment>
@@
 <net name="SDIN" class="0">
 <segment>
-<pinref part="U$1" gate="G$1" pin="SDIN"/>
-<wire x1="48.26" y1="22.86" x2="35.56" y2="22.86" width="0.1524" layer="91"/>
-<label x="35.56" y="22.86" size="1.778" layer="95"/>
+<wire x1="35.56" y1="22.86" x2="22.86" y2="22.86" width="0.1524" layer="91"/>
+<label x="22.86" y="22.86" size="1.778" layer="95"/>
+<pinref part="R9" gate="G$1" pin="2"/>
 </segment>
 <segment>
@@
 </segment>
 </net>
+<net name="N$22" class="0">
+<segment>
+<pinref part="R7" gate="G$1" pin="1"/>
+<pinref part="U$1" gate="G$1" pin="LRCLK"/>
+<wire x1="45.72" y1="27.94" x2="48.26" y2="27.94" width="0.1524" layer="91"/>
+</segment>
+</net>
+<net name="N$23" class="0">
+<segment>
+<pinref part="R8" gate="G$1" pin="1"/>
+<pinref part="U$1" gate="G$1" pin="SCLK"/>
+<wire x1="45.72" y1="25.4" x2="48.26" y2="25.4" width="0.1524" layer="91"/>
+</segment>
+</net>
+<net name="N$24" class="0">
+<segment>
+<pinref part="R9" gate="G$1" pin="1"/>
+<pinref part="U$1" gate="G$1" pin="SDIN"/>
+<wire x1="45.72" y1="22.86" x2="48.26" y2="22.86" width="0.1524" layer="91"/>
+</segment>
+</net>
