File: PCB-AMP2/AMP2.brd (EAGLE design)
At the start: 100.4 x 80 mm, 54 parts, among them IC1 LD117AS33TR, IC2 R-78E-0.5, IC3 TL77005ACD, X3 MKDSN1,5/2-5,08

Commit message: Fixed V-detect sense input.
Parts:
- moved TVS 15.3 mm to (82.5, 8.89), turned to 0 degrees
Connections:
- net +12V: no longer R3.2
- net VIN: now also R3.2
Routing:
- net +12V: track 42.0 -> 4.81 mm
- net VIN: track 3.79 -> 11.4 mm, vias 1 -> 3
Other:
- board text added: "Version: 0.2"
Changed lines of the file:
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@@
 <wire x1="55.88" y1="24.13" x2="55.88" y2="19.05" width="0.254" layer="25"/>
 <wire x1="55.88" y1="19.05" x2="60.96" y2="19.05" width="0.254" layer="25"/>
+<text x="17.78" y="67.31" size="1.778" layer="26" rot="MR0">Version: 0.2</text>
 </plain>
 <attributes>
@@
 <attribute name="VALUE" x="55.499" y="4.318" size="1.27" layer="27"/>
 </element>
-<element name="TVS" library="diode" library_urn="urn:adsk.eagle:library:210" package="SMC" package3d_urn="urn:adsk.eagle:package:43425/2" value="26Vbi" x="67.31" y="7.62" smashed="yes" rot="R270">
-<attribute name="MOUSER" value="710-824551241" x="67.31" y="7.62" size="1.778" layer="27" rot="R270" display="off"/>
-<attribute name="NAME" x="70.739" y="8.509" size="1.27" layer="25" rot="R270"/>
-<attribute name="POPULARITY" value="1" x="67.31" y="7.62" size="2.54" layer="27" rot="R270" display="off"/>
-<attribute name="VALUE" x="72.771" y="9.779" size="1.27" layer="27" rot="R270"/>
+<element name="TVS" library="diode" library_urn="urn:adsk.eagle:library:210" package="SMC" package3d_urn="urn:adsk.eagle:package:43425/2" value="26Vbi" x="82.55" y="8.89" smashed="yes">
+<attribute name="MOUSER" value="710-824551241" x="82.55" y="8.89" size="1.778" layer="27" display="off"/>
+<attribute name="NAME" x="81.661" y="12.319" size="1.27" layer="25"/>
+<attribute name="POPULARITY" value="1" x="82.55" y="8.89" size="2.54" layer="27" display="off"/>
+<attribute name="VALUE" x="80.391" y="14.351" size="1.27" layer="27"/>
 </element>
 <element name="IC3" library="linear" library_urn="urn:adsk.eagle:library:262" package="SO08" package3d_urn="urn:adsk.eagle:package:16404/2" value="TL77005ACD" x="41.91" y="21.59" smashed="yes" rot="R90">
@@
 <via x="85.471" y="14.605" extent="1-16" drill="0.35"/>
 <via x="82.931" y="12.065" extent="1-16" drill="0.35"/>
-<via x="80.391" y="9.525" extent="1-16" drill="0.35"/>
-<via x="79.121" y="6.985" extent="1-16" drill="0.35"/>
+<via x="82.931" y="13.335" extent="1-16" drill="0.35"/>
+<via x="74.041" y="6.985" extent="1-16" drill="0.35"/>
 <via x="71.501" y="5.715" extent="1-16" drill="0.35"/>
 <via x="75.311" y="5.715" extent="1-16" drill="0.35"/>
-<via x="79.121" y="5.715" extent="1-16" drill="0.35"/>
+<via x="72.771" y="5.715" extent="1-16" drill="0.35"/>
 <via x="71.501" y="6.985" extent="1-16" drill="0.35"/>
 <via x="75.311" y="6.985" extent="1-16" drill="0.35"/>
 <contactref element="L6" pad="2"/>
 <contactref element="TVS" pad="C"/>
-<contactref element="R3" pad="2"/>
-<wire x1="42.76" y1="17.78" x2="44.03" y2="16.51" width="0.3048" layer="1"/>
-<wire x1="50.8" y1="16.51" x2="51.181" y2="16.891" width="0.3048" layer="1"/>
-<wire x1="51.181" y1="16.891" x2="51.181" y2="17.78" width="0.3048" layer="1"/>
-<wire x1="51.181" y1="17.78" x2="51.435" y2="18.034" width="0.3048" layer="1"/>
-<wire x1="59.309" y1="18.034" x2="60.96" y2="19.685" width="0.3048" layer="1"/>
-<wire x1="60.96" y1="19.685" x2="60.96" y2="21.336" width="0.3048" layer="1"/>
-<wire x1="60.96" y1="21.336" x2="61.087" y2="21.463" width="0.3048" layer="1"/>
-<wire x1="61.087" y1="21.463" x2="62.992" y2="21.463" width="0.3048" layer="1"/>
-<wire x1="62.992" y1="21.463" x2="63.373" y2="21.082" width="0.3048" layer="1"/>
-<wire x1="63.373" y1="13.66143125" x2="65.71443125" y2="11.32" width="0.3048" layer="1"/>
-<wire x1="65.71443125" y1="11.32" x2="67.31" y2="11.32" width="0.3048" layer="1"/>
-<wire x1="44.03" y1="16.51" x2="50.8" y2="16.51" width="0.3048" layer="1"/>
-<wire x1="51.435" y1="18.034" x2="59.309" y2="18.034" width="0.3048" layer="1"/>
-<wire x1="63.373" y1="21.082" x2="63.373" y2="13.66143125" width="0.3048" layer="1"/>
 <via x="82.931" y="8.255" extent="1-16" drill="0.35"/>
 <via x="81.661" y="8.255" extent="1-16" drill="0.35"/>
@@
 <via x="81.661" y="9.525" extent="1-16" drill="0.35"/>
 <via x="82.931" y="9.525" extent="1-16" drill="0.35"/>
-<via x="80.391" y="8.255" extent="1-16" drill="0.35"/>
+<via x="74.041" y="5.715" extent="1-16" drill="0.35"/>
 <via x="81.661" y="10.795" extent="1-16" drill="0.35"/>
-<via x="80.391" y="6.985" extent="1-16" drill="0.35"/>
+<via x="72.771" y="6.985" extent="1-16" drill="0.35"/>
 <via x="81.661" y="6.985" extent="1-16" drill="0.35"/>
 </signal>
@@
 <wire x1="33.02" y1="9.0631" x2="32.9989" y2="9.042" width="2.032" layer="16"/>
 <contactref element="D1" pad="A"/>
+<contactref element="R3" pad="2"/>
+<wire x1="42.76" y1="17.78" x2="43.9058" y2="16.6342" width="0.4064" layer="1"/>
+<wire x1="43.9058" y1="16.6342" x2="44.45" y2="16.6342" width="0.4064" layer="1"/>
+<via x="44.45" y="16.6342" extent="1-16" drill="0.35"/>
+<wire x1="44.45" y1="16.6342" x2="44.45" y2="12.7" width="0.4064" layer="16"/>
+<wire x1="44.45" y1="12.7" x2="44.069" y2="12.319" width="0.4064" layer="16"/>
+<wire x1="44.069" y1="12.319" x2="43.053" y2="12.319" width="0.4064" layer="16"/>
+<via x="43.053" y="12.319" extent="1-16" drill="0.35"/>
 </signal>
 <signal name="N$14">
